File: eagle/main.brd (EAGLE design)
At the start: 55 x 127 mm, 81 parts, among them IC1 LD117AS50TR, IC2 LD117AS33TR, IC3 OPA340U, Q1 BSS138, T1 FDV304P, U1 STM32F777VIT, U2 RFM26W, U3 PAM8302, U4 MICROSD-PUSH-OUT, X1 16MHz, X2 SMA

Commit message: Add files via upload
Parts:
- R5: value 47k -> 1k
Changed lines of the file:
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@@
 <element name="R3" library="rcl" package="R0805" value="9k1" x="20.955" y="105.41" rot="R180"/>
 <element name="R4" library="rcl" package="R0805" value="1k" x="26.035" y="105.41" rot="R180"/>
-<element name="R5" library="rcl" package="R0805" value="47k" x="39.37" y="109.855"/>
+<element name="R5" library="rcl" package="R0805" value="1k" x="39.37" y="109.855"/>
 <element name="R6" library="rcl" package="R1206" value="22R" x="42.545" y="113.665" rot="R180"/>
 <element name="R7" library="resistor" package="R0805" value="680R" x="9.525" y="11.43"/>

Commit message: Add files via upload
Parts:
- moved R7 0.32 mm to (9.53, 11.7), turned to 180 degrees
Connections:
- net ADC1_0: now also R7.2; no longer R7.1, R8.2
- net N$4: now also R7.1, R8.2; no longer R7.2
Routing:
- net N$4: track 2.60 -> 6.86 mm
- net ADC1_0: track 51.3 -> 48.4 mm
- net GND: vias 409 -> 425
Changed lines of the file:
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@@
 <element name="R5" library="rcl" package="R0805" value="1k" x="39.37" y="109.855"/>
 <element name="R6" library="rcl" package="R1206" value="22R" x="42.545" y="113.665" rot="R180"/>
-<element name="R7" library="resistor" package="R0805" value="680R" x="9.525" y="11.43"/>
+<element name="R7" library="resistor" package="R0805" value="680R" x="9.525" y="11.7475" rot="R180"/>
 <element name="R8" library="resistor" package="R0805" value="22R" x="9.525" y="8.89" rot="R180"/>
 <element name="R9" library="resistor" package="R0805" value="47k" x="20.955" y="13.97" rot="R270"/>
@@
 <via x="10.795" y="10.16" extent="1-16" drill="0.2"/>
 <via x="13.97" y="10.16" extent="1-16" drill="0.2"/>
-<via x="9.525" y="10.16" extent="1-16" drill="0.2"/>
+<via x="43.65625" y="77.1525" extent="1-16" drill="0.2"/>
 <via x="15.875" y="18.415" extent="1-16" drill="0.2"/>
 <via x="19.05" y="18.415" extent="1-16" drill="0.2"/>
@@
 <wire x1="32.385" y1="42.13" x2="32.385" y2="41.275" width="0.254" layer="1"/>
 <wire x1="32.385" y1="41.275" x2="31.75" y2="40.64" width="0.254" layer="1"/>
+<via x="43.815" y="81.12125" extent="1-16" drill="0.2"/>
+<via x="43.815" y="82.2325" extent="1-16" drill="0.2"/>
+<via x="43.02125" y="83.5025" extent="1-16" drill="0.2"/>
+<via x="41.75125" y="83.5025" extent="1-16" drill="0.2"/>
+<via x="40.79875" y="84.61375" extent="1-16" drill="0.2"/>
+<via x="39.52875" y="85.88375" extent="1-16" drill="0.2"/>
+<via x="38.57625" y="83.34375" extent="1-16" drill="0.2"/>
+<via x="36.98875" y="83.34375" extent="1-16" drill="0.2"/>
+<via x="35.71875" y="83.34375" extent="1-16" drill="0.2"/>
+<via x="35.08375" y="82.39125" extent="1-16" drill="0.2"/>
+<via x="35.08375" y="81.12125" extent="1-16" drill="0.2"/>
+<via x="39.52875" y="82.07375" extent="1-16" drill="0.2"/>
+<via x="39.52875" y="80.48625" extent="1-16" drill="0.2"/>
+<via x="41.11625" y="80.16875" extent="1-16" drill="0.2"/>
+<via x="30.63875" y="85.56625" extent="1-16" drill="0.2"/>
+<via x="34.44875" y="84.93125" extent="1-16" drill="0.2"/>
 </signal>
 <signal name="+3V3" class="1">
@@
 <contactref element="U1" pad="22"/>
 <contactref element="IC3" pad="6"/>
-<contactref element="R7" pad="1"/>
-<contactref element="R8" pad="2"/>
-<wire x1="8.5725" y1="11.43" x2="8.5725" y2="8.89" width="0.127" layer="1"/>
-<wire x1="8.5725" y1="8.89" x2="8.575" y2="8.89" width="0.127" layer="1"/>
-<wire x1="8.5725" y1="11.43" x2="8.575" y2="11.43" width="0.127" layer="1"/>
 <wire x1="29.2735" y1="39.9415" x2="29.2735" y2="40.4495" width="0.127" layer="1"/>
 <wire x1="33.2105" y1="36.0045" x2="29.2735" y2="39.9415" width="0.127" layer="1"/>
@@
 <wire x1="12.065" y1="19.1262" x2="12.065" y2="19.558" width="0.127" layer="1"/>
 <wire x1="29.2735" y1="40.4495" x2="29.265" y2="40.51" width="0.127" layer="1"/>
-<wire x1="8.636" y1="15.24" x2="8.636" y2="11.43" width="0.127" layer="1"/>
+<wire x1="8.636" y1="15.24" x2="8.636" y2="12.065" width="0.127" layer="1"/>
 <wire x1="12.065" y1="18.669" x2="8.636" y2="15.24" width="0.127" layer="1"/>
 <wire x1="12.065" y1="19.1262" x2="12.065" y2="18.669" width="0.127" layer="1"/>
-<wire x1="8.636" y1="11.43" x2="8.575" y2="11.43" width="0.127" layer="1"/>
+<contactref element="R7" pad="2"/>
+<wire x1="8.636" y1="12.065" x2="8.575" y2="12.065" width="0.4064" layer="1"/>
+<wire x1="8.575" y1="12.065" x2="8.575" y2="11.7475" width="0.4064" layer="1"/>
 </signal>
 <signal name="LED_RED">
@@
 <wire x1="50.8" y1="117.475" x2="48" y2="124.4346" width="1.016" layer="1" curve="-37.251813"/>
 </signal>
-<signal name="N$4">
-<contactref element="R7" pad="2"/>
-<contactref element="IC3" pad="2"/>
-<wire x1="10.4775" y1="13.5255" x2="10.4775" y2="11.43" width="0.127" layer="1"/>
-<wire x1="10.795" y1="13.843" x2="10.4775" y2="13.5255" width="0.127" layer="1"/>
-<wire x1="10.4775" y1="11.43" x2="10.475" y2="11.43" width="0.127" layer="1"/>
-<wire x1="10.795" y1="13.843" x2="10.795" y2="13.8938" width="0.127" layer="1"/>
-</signal>
 <signal name="N$5">
 <contactref element="C22" pad="1"/>
@@
 <wire x1="15.875" y1="15.3035" x2="15.875" y2="15.37" width="0.127" layer="1"/>
 </signal>
+<signal name="N$4">
+<contactref element="R8" pad="2"/>
+<wire x1="8.5725" y1="10.4775" x2="8.5725" y2="8.89" width="0.127" layer="1"/>
+<wire x1="8.5725" y1="8.89" x2="8.575" y2="8.89" width="0.127" layer="1"/>
+<contactref element="R7" pad="1"/>
+<contactref element="IC3" pad="2"/>
+<wire x1="10.795" y1="13.8938" x2="10.795" y2="12.0675" width="0.4064" layer="1"/>
+<wire x1="10.795" y1="12.0675" x2="10.475" y2="11.7475" width="0.4064" layer="1"/>
+<wire x1="8.5725" y1="10.4775" x2="8.73125" y2="10.63625" width="0.127" layer="1"/>
+<wire x1="8.73125" y1="10.63625" x2="10.31875" y2="10.63625" width="0.127" layer="1"/>
+<wire x1="10.31875" y1="10.63625" x2="10.4775" y2="10.795" width="0.127" layer="1"/>
+<wire x1="10.4775" y1="10.795" x2="10.4775" y2="11.745" width="0.127" layer="1"/>
+<wire x1="10.4775" y1="11.745" x2="10.475" y2="11.7475" width="0.127" layer="1"/>
+</signal>
 </signals>

Commit message: Add files via upload
Parts:
- added C0: 8p2, rcl:C0805
- added C34: 10n, rcl:C0805
- added CC1, CC2, CC3: 1000p, rcl:C0805
- added CM: 13p, rcl:C0805
- added CM1, CM2, CM3: 9p1, rcl:C0805
- added CR1: 3p9, rcl:C0805
- added CR2: 2p2, rcl:C0805
- added L0: 30nH, resistor:R0805
- added LCHOKE: 220nH, resistor:R0805
- added LM1: 27nH, resistor:R0805
- added LM2: 22nH, resistor:R0805
- added LM3: 15nH, resistor:R0805
- added LR1: 56nH, resistor:R0805
- added LR2: 51nH, resistor:R0805
- added U5: SI4463-C2A-GM, SI4463-C2A-GM:QFN50P400X400X90-20N
- added X3: ILSI 32MHz TCXO, ILSI_tcxo:ASE
- U2: value RFM26W -> CG2179M2; device hoperf:MODULE_16X16_16PIN -> CG2179M2:SOT363
- moved U2 222.4 mm to (-9.53, -115.9)
Connections:
- removed net N$3: U2.1, X2.1
- new net 32M: U5.17, X3.3
- new net N$21: CM3.1, LM3.2, X2.1
- new net N$22: CC2.2, CM2.1, LM3.1
- new net N$23: C0.2, L0.1
- new net N$24: CM.1, L0.2, LM1.1
- new net N$25: CM1.1, LM1.2, LM2.1
- new net N$26: CC3.1, LM2.2
- new net N$29: CC1.1, CR2.2, LR2.2
- new net N$30: CC3.2, U2.1
- new net N$31: CC1.2, U2.3
- new net N$32: CC2.1, U2.5
- new net RXN: CR1.1, LR1.1, LR2.1, U5.3
- new net RXP: CR2.1, LR1.2, U5.2
- new net TX: C0.1, LCHOKE.1, U5.4
- net +3V3: now also C34.1, LCHOKE.2, U5.6, U5.8, X3.4; no longer U2.5
- net GND: now also C34.2, CM.2, CM1.2, CM2.2, CM3.2, CR1.2, U5.18, U5.21, X3.2; no longer U2.16
- net SPI1_CS: now also U5.15; no longer U2.13
- net SPI1_MISO: now also U5.13; no longer U2.10
- net SPI1_MOSI: now also U5.14; no longer U2.11
- net SPI1_SCK: now also U5.12; no longer U2.12
- net TRX_NIRQ: now also U5.11; no longer U2.14
- net TRX_RX_SW: no longer U2.3
- net TRX_SDN: now also U5.1; no longer U2.15
- net TRX_TX_SW: no longer U2.4
Routing:
- net N$3: track 18.9 -> 0.00 mm
- net N$21: track 0.00 -> 18.8 mm

Commit message: Add files via upload
Parts:
- removed C24, C25, C27: 220p, rcl:C1206
- removed L3, L4: (no value), inductor-neosid:SM-B5
- removed U3: PAM8302, pam:SOP65P490X110-8N
- added IC4: L272D, linear:SO08
- added Q2: BSS138, bss138_10:SOT23
- added R19, R20, R23, R24: 10k, resistor:R0805
- added R21, R22, R25: 22k, resistor:R0805
- R13, R14: value 10k -> 4k7
- R7: value 680R -> 820R
Connections:
- removed net +UB: C8.+, IC1.3, JP2.2, R3.2
- removed net SPK_INT_N: C25.1, JP4.2, L4.2
- removed net SPK_INT_P: C24.2, JP4.1, L3.2
- new net +BATT: C32.1, C8.+, IC1.3, JP2.2, L5.1, R14.1, R3.2
- new net N$27: IC4.6, R22.2
- new net N$28: IC4.5, R23.2, R24.1
- new net N$3: IC4.8, R19.1, R20.2
- new net N$33: IC4.3, JP4.1, R24.2
- net +5V: no longer C32.1, L5.1
- net GND: now also C30.1, IC4.4, Q2.2, R13.2; no longer C24.1, C25.2, C27.2, C30.2, R14.1, U3.7
- net N$13: now also C30.2, R13.1, R14.2, R21.1, R22.1, R25.1; no longer L4.1, U3.8
- net N$14: now also Q2.3, R19.2, R25.2; no longer C27.1, U3.3
- net N$15: now also IC4.7, R21.2; no longer C30.1, R13.1, R14.2, U3.4
- net N$8: now also IC4.2; no longer R13.2, U3.6
- net N$9: now also IC4.1, JP4.2, R20.1, R23.1; no longer L3.1, U3.5
- net SPK_SDN: now also Q2.1; no longer U3.1
Routing:
- net +BATT: track 0.00 -> 15.3 mm
- net +UB: track 11.7 -> 0.00 mm
- net SPK_INT_P: track 9.98 -> 0.00 mm
- net SPK_INT_N: track 9.98 -> 0.00 mm
- net N$15: track 7.26 -> 0.00 mm
- net +5V: track 142.6 -> 138.9 mm
- net N$9: track 2.62 -> 0.00 mm
- net N$13: track 2.62 -> 0.00 mm
- net GND: track 14.9 -> 13.1 mm, vias 425 -> 424
- net N$8: track 13.9 -> 13.0 mm

Commit message: Add files via upload
Parts:
- removed IC4: L272D, linear:SO08
- removed R21, R22: 22k, resistor:R0805
- added U3: L272, L272:SO16
- C26: value 1u -> 470n
- R20: value 10k -> 15k
Connections:
- removed net N$15: IC4.7, R21.2
- removed net N$28: IC4.5, R23.2, R24.1
- removed net N$33: IC4.3, JP4.1, R24.2
- removed net N$8: C29.1, C31.1, IC4.2, L5.2
- removed net N$9: IC4.1, JP4.2, R20.1, R23.1
- new net PA_SUPP: C29.1, C31.1, L5.2, U3.4
- new net SPK_N: JP4.2, R20.2, R24.2, U3.3
- new net SPK_P: JP4.1, R23.2, U3.5
- net GND: now also U3.6; no longer IC4.4
- net N$13: now also R23.1, R24.1, U3.11; no longer C30.2, R13.1, R14.2, R21.1, R22.1, R25.1
- net N$27: now also C30.2, R13.1, R14.2, R25.1, U3.12, U3.13; no longer IC4.6, R22.2
- net N$3: now also R20.1, U3.14; no longer IC4.8, R20.2
Routing:
- net PA_SUPP: track 0.00 -> 13.0 mm
- net N$8: track 13.0 -> 0.00 mm

Commit message: Add files via upload
Parts:
- removed JP9: ACC_CONN, pinhead:1X04
- added U$1: ADXL345, adxl345:LGA14
Connections:
- net +3V3: now also U$1.P$1, U$1.P$7; no longer JP9.1
- net GND: now also U$1.P$12, U$1.P$2, U$1.P$4, U$1.P$5, U$1.P$6; no longer JP9.4
- net I2C1_SCL: now also U$1.P$14; no longer JP9.2
- net I2C1_SDA: now also U$1.P$13; no longer JP9.3
Routing:
- net I2C1_SCL: track 19.5 -> 13.7 mm
- net I2C1_SDA: track 17.4 -> 13.0 mm
Changed lines of the file:
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@@
 <element name="JP7" library="pinhead" package="1X03" value="DBG_CONN" x="2.54" y="45.085" rot="R270"/>
 <element name="JP8" library="pinhead" package="1X03" value="KBD_CONN" x="46.99" y="49.53" rot="R90"/>
-<element name="JP9" library="pinhead" package="1X04" value="ACC_CONN" x="6.35" y="36.195"/>
 <element name="L1" library="inductor-neosid" package="SM-B5" value="" x="22.86" y="34.925">
 <attribute name="MPN" value="" x="22.86" y="34.925" size="1.778" layer="27" display="off"/>
@@
 <element name="R25" library="resistor" package="R0805" value="22k" x="-25.4" y="-157.1625"/>
 <element name="U3" library="L272" package="SO16" value="L272" x="-33.02" y="-153.67"/>
+<element name="U$1" library="adxl345" package="LGA14" value="ADXL345" x="-44.7675" y="-154.6225"/>
 </elements>
 <signals>
@@
 <contactref element="JP6" pad="3"/>
 <contactref element="JP8" pad="3"/>
-<contactref element="JP9" pad="4"/>
 <contactref element="JP7" pad="3"/>
 <polygon width="0.4064" layer="1" isolate="0.254" orphans="yes">
@@
 <contactref element="Q2" pad="2"/>
 <contactref element="U3" pad="6"/>
+<contactref element="U$1" pad="P$6"/>
+<contactref element="U$1" pad="P$5"/>
+<contactref element="U$1" pad="P$4"/>
+<contactref element="U$1" pad="P$2"/>
+<contactref element="U$1" pad="P$12"/>
+<wire x1="-45.8675" y1="-155.8225" x2="-45.8675" y2="-156.6225" width="0" layer="19" extent="1-1"/>
+<wire x1="-45.8675" y1="-155.0225" x2="-45.8675" y2="-155.8225" width="0" layer="19" extent="1-1"/>
+<wire x1="-45.8675" y1="-153.4225" x2="-45.8675" y2="-155.0225" width="0" layer="19" extent="1-1"/>
+<wire x1="-43.6675" y1="-153.4225" x2="-45.8675" y2="-153.4225" width="0" layer="19" extent="1-1"/>
+<wire x1="-31.115" y1="-156.7434" x2="-43.6675" y2="-153.4225" width="0" layer="19" extent="1-1"/>
 <wire x1="-23.18" y1="-116.2525" x2="-31.115" y2="-156.7434" width="0" layer="19" extent="1-1"/>
 <wire x1="-9.525" y1="-116.7875" x2="-23.18" y2="-116.2525" width="0" layer="19" extent="1-1"/>
@@
 <wire x1="5.715" y1="45.085" x2="2.54" y2="42.545" width="0" layer="19" extent="1-1"/>
 <wire x1="13.97" y1="37.465" x2="13.335" y2="41.91" width="0" layer="19" extent="1-1"/>
-<wire x1="10.16" y1="36.195" x2="13.97" y2="37.465" width="0" layer="19" extent="1-1"/>
 <wire x1="31.75" y1="13.335" x2="27.305" y2="12.065" width="0" layer="19" extent="1-1"/>
 <wire x1="34.925" y1="13.335" x2="31.75" y2="13.335" width="0" layer="19" extent="1-1"/>
@@
 <contactref element="JP6" pad="1"/>
 <contactref element="JP8" pad="1"/>
-<contactref element="JP9" pad="1"/>
 <wire x1="23.1775" y1="6.4135" x2="23.1775" y2="5.715" width="0.5" layer="1"/>
 <wire x1="24.3205" y1="7.5565" x2="23.1775" y2="6.4135" width="0.5" layer="1"/>
@@
 <wire x1="17.2085" y1="34.925" x2="20.86" y2="34.925" width="0.5" layer="1"/>
 <wire x1="17.2085" y1="34.925" x2="17.145" y2="34.25" width="0.5" layer="1"/>
-<wire x1="2.667" y1="36.195" x2="2.54" y2="36.195" width="0.5" layer="1"/>
 <wire x1="4.572" y1="34.29" x2="2.667" y2="36.195" width="0.5" layer="1"/>
 <wire x1="16.8275" y1="34.29" x2="9.0805" y2="34.29" width="0.5" layer="1"/>
@@
 <contactref element="U5" pad="6"/>
 <contactref element="LCHOKE" pad="2"/>
-<wire x1="43.8785" y1="106.3625" x2="44.1325" y2="106.553" width="0" layer="19" extent="1-1"/>
+<contactref element="U$1" pad="P$1"/>
+<contactref element="U$1" pad="P$7"/>
+<wire x1="-44.7675" y1="-156.7225" x2="-45.8675" y2="-152.6225" width="0" layer="19" extent="1-1"/>
+<wire x1="-8.2575" y1="-24.4475" x2="-45.8675" y2="-152.6225" width="0" layer="19" extent="1-1"/>
+<wire x1="-8.255" y1="-11.4325" x2="-8.2575" y2="-24.4475" width="0" layer="19" extent="1-1"/>
+<wire x1="-6.5975" y1="-11.3825" x2="-8.255" y2="-11.4325" width="0" layer="19" extent="1-1"/>
+<wire x1="-3.8575" y1="-8.6025" x2="-6.5975" y2="-11.3825" width="0" layer="19" extent="1-1"/>
+<wire x1="-2.8575" y1="-8.6025" x2="-3.8575" y2="-8.6025" width="0" layer="19" extent="1-1"/>
+<wire x1="12.954" y1="2.54" x2="-2.8575" y2="-8.6025" width="0" layer="19" extent="1-1"/>
+<wire x1="17.015" y1="42.26" x2="17.018" y2="42.26" width="0" layer="19" extent="1-1"/>
+<wire x1="18.7325" y1="56.0705" x2="18.765" y2="56.01" width="0" layer="19" extent="1-1"/>
 <wire x1="32.515" y1="54.26" x2="32.5755" y2="54.2925" width="0" layer="19" extent="1-1"/>
-<wire x1="18.765" y1="56.01" x2="18.7325" y2="56.0705" width="0" layer="19" extent="1-1"/>
-<wire x1="17.018" y1="42.26" x2="17.015" y2="42.26" width="0" layer="19" extent="1-1"/>
-<wire x1="-2.8575" y1="-8.6025" x2="12.954" y2="2.54" width="0" layer="19" extent="1-1"/>
-<wire x1="-3.8575" y1="-8.6025" x2="-2.8575" y2="-8.6025" width="0" layer="19" extent="1-1"/>
-<wire x1="-6.5975" y1="-11.3825" x2="-3.8575" y2="-8.6025" width="0" layer="19" extent="1-1"/>
-<wire x1="-8.255" y1="-11.4325" x2="-6.5975" y2="-11.3825" width="0" layer="19" extent="1-1"/>
-<wire x1="-8.2575" y1="-24.4475" x2="-8.255" y2="-11.4325" width="0" layer="19" extent="1-1"/>
+<wire x1="44.1325" y1="106.553" x2="43.8785" y2="106.3625" width="0" layer="19" extent="1-1"/>
 </signal>
 <signal name="SWDIO">
@@
 <signal name="I2C1_SDA">
 <contactref element="U1" pad="93"/>
-<contactref element="JP9" pad="3"/>
 <wire x1="12.7635" y1="45.7835" x2="16.9545" y2="45.7835" width="0.127" layer="1"/>
 <wire x1="12.5095" y1="46.0375" x2="12.7635" y2="45.7835" width="0.127" layer="1"/>
@@
 <wire x1="10.7315" y1="45.7835" x2="10.9855" y2="46.0375" width="0.127" layer="1"/>
 <wire x1="10.7315" y1="39.3065" x2="10.7315" y2="45.7835" width="0.127" layer="1"/>
-<wire x1="7.62" y1="36.195" x2="10.7315" y2="39.3065" width="0.127" layer="1"/>
 <wire x1="16.9545" y1="45.7835" x2="17.015" y2="45.76" width="0.127" layer="1"/>
+<contactref element="U$1" pad="P$13"/>
+<wire x1="10.7315" y1="39.3065" x2="-43.6675" y2="-152.6225" width="0" layer="19" extent="1-1"/>
 </signal>
 <signal name="I2C1_SCL">
 <contactref element="U1" pad="92"/>
-<contactref element="JP9" pad="2"/>
 <wire x1="9.3345" y1="46.2915" x2="16.9545" y2="46.2915" width="0.127" layer="1"/>
 <wire x1="5.08" y1="42.037" x2="9.3345" y2="46.2915" width="0.127" layer="1"/>
-<wire x1="5.08" y1="36.195" x2="5.08" y2="42.037" width="0.127" layer="1"/>
 <wire x1="16.9545" y1="46.2915" x2="17.015" y2="46.26" width="0.127" layer="1"/>
+<contactref element="U$1" pad="P$14"/>
+<wire x1="5.08" y1="42.037" x2="-44.7675" y2="-152.5225" width="0" layer="19" extent="1-1"/>
 </signal>
 <signal name="USART2_RX">

Commit message: Add files via upload
Parts:
- added D1: CGRM4007-G, diode:SOD-123_MINI-SMA
- added U$2: 2A, chiptron_cz:1206
- C10, C12, C13, C14, C15, C16, C17, C18: device resistor:SMC_C -> resistor:C1206
- JP2: device pinhead:1X02 -> pinhead:1X03/90
- U4: value MICROSD-PUSH-OUT -> ADAM TECH MCSP-Q1-08-A-SG
- moved U4 34.3 mm to (75.9, 77.2), turned to 90 degrees
Connections:
- new net N$8: JP2.3, U$2.1
- net +3V3: now also C10.1, C12.1, C13.1, C14.1, C15.1, C16.1, C17.1, C18.1; no longer C10.+, C12.+, C13.+, C14.+, C15.+, C16.+, C17.+, C18.+
- net +BATT: now also D1.C; no longer JP2.2
- net GND: now also C10.2, C12.2, C13.2, C14.2, C15.2, C16.2, C17.2, C18.2, D1.A; no longer C10.-, C12.-, C13.-, C14.-, C15.-, C16.-, C17.-, C18.-
- net SPI1_CS: now also JP3.10; no longer U5.15
- net SPI1_MISO: no longer U5.13
- net SPI1_MOSI: now also JP3.8; no longer U5.14
- net SPI1_SCK: now also JP3.9; no longer U5.12
- net SPI2_CS: now also U5.15; no longer JP3.10
- net SPI2_MISO: now also U5.13
- net SPI2_MOSI: now also U5.14; no longer JP3.8
- net SPI2_SCK: now also U5.12; no longer JP3.9
Routing:
- net +3V3: track 377.5 -> 0.00 mm, vias 8 -> 0
- net +5V: track 138.9 -> 0.00 mm, vias 4 -> 0
- net TRX_RX_SW: track 98.0 -> 0.00 mm, vias 4 -> 0
- net LED_RED: track 89.6 -> 0.00 mm, vias 2 -> 0
- net SD_CMD: track 87.9 -> 0.00 mm
- net TRX_TX_SW: track 84.3 -> 0.00 mm, vias 2 -> 0
- net ADC2_3: track 83.7 -> 0.00 mm, vias 2 -> 0
- net TFT_A0: track 83.2 -> 0.00 mm, vias 3 -> 0
- net LED_GRN: track 81.4 -> 0.00 mm, vias 2 -> 0
- net SPI2_CS: track 81.1 -> 0.00 mm, vias 4 -> 0
- net SPI2_SCK: track 76.8 -> 0.00 mm, vias 3 -> 0
- net SPI2_MOSI: track 75.7 -> 0.00 mm, vias 5 -> 0
- net BLIGHT_CTRL: track 73.4 -> 0.00 mm, vias 4 -> 0
- net TFT_RST: track 70.0 -> 0.00 mm, vias 5 -> 0
- net SPI1_SCK: track 69.6 -> 0.00 mm, vias 4 -> 0
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Other:
- board text added: "TR_9_MAIN_BOARD_1.1"
- board text removed: "TR_9_MAIN_BOARD_1.0"

Commit message: Add files via upload
Parts:
- added R21, R22: 4k7, rcl:R0805
- moved D1 281.2 mm to (23.2, 102.9)
- moved U$2 269.1 mm to (17.5, 98.1), flipped to the bottom, turned to 270 degrees
- moved U$1 201.2 mm to (9.84, 39.1)
- moved U4 24.9 mm to (51.1, 79.7)
- moved JP2 6.35 mm to (23.5, 95.9), flipped to the bottom
- moved IC1 3.81 mm to (23.5, 88.3)
- moved IC2 3.81 mm to (23.5, 78.1)
- moved C9 2.54 mm to (28.6, 88.3)
- moved C8 2.54 mm to (23.5, 95.9)
- moved R1 0.90 mm to (11.4, 45.7)
Connections:
- net +3V3: now also R21.2, R22.2
- net +BATT: now also U$2.2
- net GND: now also JP2.3; no longer JP2.1
- net I2C1_SCL: now also R22.1
- net I2C1_SDA: now also R21.1
- net N$8: now also JP2.1; no longer JP2.3
