File: eagle/main.brd (EAGLE design)
At the start: 55 x 127 mm, 106 parts, among them IC1 LD117AS50TR, IC2 LD117AS33TR, IC3 OPA340U, Q1 BSS138, Q2 BSS138, T1 FDV304P, U1 STM32F777VIT, U2 CG2179M2, U3 L272, U4 ADAM TECH MCSP-Q1-08-A-SG, U5 SI4463-C2A-GM, X1 16MHz, X2 SMA, X3 ILSI 32MHz TCXO

Commit message: Add files via upload
Parts:
- added C24, C25: 10n, resistor:C0805
- C26, C32: device rcl:C1206 -> rcl:C0805
- moved U2 228.5 mm to (48.6, 105.1), turned to 270 degrees
- moved CM 220.1 mm to (41.0, 103.5), turned to 180 degrees
- moved CC3 219.3 mm to (46.7, 107.3)
- moved CC1 209.2 mm to (47.6, 102.2), turned to 90 degrees
- moved CC2 208.3 mm to (51.1, 106.0), turned to 90 degrees
- moved C0 193.9 mm to (41.0, 99.7), turned to 180 degrees
- moved CM1 193.9 mm to (41.0, 105.4), turned to 180 degrees
- moved R25 193.5 mm to (42.2, 24.1), turned to 180 degrees
- moved R24 186.1 mm to (42.2, 22.2), turned to 180 degrees
- moved U3 185.4 mm to (41.3, 16.2)
- moved CR2 183.9 mm to (47.6, 98.7), turned to 90 degrees
- moved CM2 183.5 mm to (50.2, 108.9), turned to 180 degrees
- moved CM3 183.5 mm to (50.2, 114.6), turned to 180 degrees
- moved CR1 179.2 mm to (43.8, 100.6), turned to 90 degrees
- moved R23 177.3 mm to (48.3, 16.2), turned to 270 degrees
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Connections:
- net +3V3: now also C24.1, C25.1
- net GND: now also C24.2, C25.2
- net TRX_RX_SW: now also U2.4
- net TRX_TX_SW: now also U2.6
Routing:
- net +3V3: track 0.00 -> 332.9 mm, vias 0 -> 9
- net +BATT: track 0.00 -> 123.7 mm, vias 0 -> 3
- net TRX_RX_SW: track 0.00 -> 88.8 mm, vias 0 -> 2
- net SPI1_SCK: track 0.00 -> 81.9 mm, vias 0 -> 2
- net SPI1_MOSI: track 0.00 -> 80.4 mm, vias 0 -> 2
- net ADC2_3: track 0.00 -> 79.7 mm, vias 0 -> 2
- net TRX_TX_SW: track 0.00 -> 77.6 mm, vias 0 -> 4
- net SPI1_CS: track 0.00 -> 75.9 mm, vias 0 -> 2
- net LED_GRN: track 0.00 -> 75.2 mm, vias 0 -> 2
- net LED_RED: track 0.00 -> 73.3 mm, vias 0 -> 2
- net TRX_SDN: track 0.00 -> 67.3 mm, vias 0 -> 2
- net TFT_A0: track 0.00 -> 67.2 mm, vias 0 -> 2
- net TFT_RST: track 0.00 -> 66.2 mm, vias 0 -> 2
- net BLIGHT_CTRL: track 0.00 -> 62.1 mm, vias 0 -> 2
- net PTT_INT: track 0.00 -> 56.9 mm, vias 0 -> 2
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
Commit message: Add files via upload
Routing:
- net +3V3: track 332.9 -> 354.1 mm, vias 9 -> 12
- net GND: track 0.00 -> 15.6 mm, vias 0 -> 124
- net I2C1_SCL: track 21.7 -> 16.3 mm
- net N$25: track 1.91 -> 5.30 mm, vias 0 -> 5
- net USART2_RX: track 19.3 -> 16.0 mm
- net USART2_TX: track 17.8 -> 15.2 mm
- net TX: track 1.91 -> 4.10 mm
- net N$32: track 0.00 -> 1.64 mm

Commit message: Add files via upload
Routing:
- net +3V3: track 354.1 -> 367.5 mm, vias 12 -> 14
- net GND: track 15.6 -> 18.2 mm, vias 124 -> 562
- net DAC_OUT: track 20.0 -> 20.9 mm

Commit message: Add files via upload
Connections:
- net +3V3: now also U$1.P$6
- net GND: no longer U$1.P$6
Routing:
- net +3V3: track 367.5 -> 368.7 mm
Changed lines of the file:
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@@
 </class>
 </classes>
-<designrules name="Moje Technoservice 2">
+<designrules name="Moje Technoservice 2 *">
 <description language="de">&lt;b&gt;EAGLE Design Rules&lt;/b&gt;
 &lt;p&gt;
@@
 <param name="mlMinCreamFrame" value="0mil"/>
 <param name="mlMaxCreamFrame" value="0mil"/>
-<param name="mlViaStopLimit" value="0mil"/>
+<param name="mlViaStopLimit" value="0.3mm"/>
 <param name="srRoundness" value="0"/>
 <param name="srMinRoundness" value="0mil"/>
@@
 <contactref element="Q2" pad="2"/>
 <contactref element="U3" pad="6"/>
-<contactref element="U$1" pad="P$6"/>
 <contactref element="U$1" pad="P$5"/>
 <contactref element="U$1" pad="P$4"/>
@@
 <wire x1="40.3225" y1="93.98" x2="40.3225" y2="95.6945" width="0.3" layer="1"/>
 <wire x1="40.3225" y1="95.6945" x2="40.1955" y2="95.8215" width="0.3" layer="1"/>
+<contactref element="U$1" pad="P$6"/>
+<wire x1="8.7425" y1="37.0525" x2="9.8425" y2="37.0525" width="0.4064" layer="1"/>
+<wire x1="9.8425" y1="37.0525" x2="9.8425" y2="36.9525" width="0.4064" layer="1"/>
 </signal>
 <signal name="SWDIO">

Commit message: Add files via upload
Parts:
- moved U4 49.1 mm to (2.86, 56.5), turned to 270 degrees
- moved R2 18.4 mm to (12.5, 76.9)
- moved JP7 17.9 mm to (20.3, 46.7)
- moved JP1 14.8 mm to (8.89, 74.3)
Connections:
- net +3V3: now also U4.4; no longer U4.5
- net GND: now also U4.6; no longer U4.3
- net SD_CLK: now also U4.5; no longer U4.4
- net SD_CMD: now also U4.3; no longer U4.6
- net SD_D0: now also U4.7; no longer U4.2
- net SD_D1: now also U4.8; no longer U4.1
- net SD_D2: now also U4.1; no longer U4.8
- net SD_D3: now also U4.2; no longer U4.7
Routing:
- net SD_CLK: track 55.4 -> 11.0 mm
- net SWDIO: track 22.2 -> 57.3 mm, vias 0 -> 2
- net SD_CMD: track 46.5 -> 11.5 mm, vias 2 -> 0
- net SD_D3: track 34.2 -> 7.93 mm, vias 2 -> 0
- net SD_D2: track 28.7 -> 3.57 mm, vias 4 -> 0
- net USART2_RX: track 16.0 -> 4.17 mm
- net USART2_TX: track 15.2 -> 3.35 mm
- net NRST: track 35.8 -> 45.4 mm, vias 1 -> 3
- net +3V3: track 368.7 -> 360.7 mm, vias 14 -> 15
- net SWCLK: track 17.6 -> 25.3 mm, vias 0 -> 2
- net SD_D1: track 23.3 -> 26.5 mm, vias 0 -> 2
- net +BATT: track 123.7 -> 121.7 mm
- net N$25: track 5.30 -> 6.57 mm, vias 5 -> 4
- net SD_D0: track 28.0 -> 29.1 mm
- net LED_RED: track 73.3 -> 73.9 mm
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
Commit message: Add files via upload
Parts:
- removed C1, C3: 18p, rcl:C0805
- removed C11: 10u, resistor:C1206
- removed C17: 22u/TA, resistor:C1206
- removed JP3: TFT_CONN, pinhead:1X16
- removed Q2: BSS138, bss138_10:SOT23
- removed R5: 1k, rcl:R0805
- removed R6: 22R, rcl:R1206
- removed T1: FDV304P, FDV304P:SOT23-3
- removed U2: CG2179M2, CG2179M2:SOT363
- added C27, C35, C38, C42: 10p, rcl:C0805
- added C37, C47: 100p, rcl:C0805
- added C39: 12p, rcl:C0805
- added C40: 7p, rcl:C0805
- added C41, C48: 1000p, rcl:C0805
- added C43: 2p, rcl:C0805
- added C45, C46: 1u/TA, resistor:C1206
- added C_ACG: 33p, rcl:C0805
- added L3: 2.7nH, rcl:R0805
- added L4, L6: 1nH, resistor:R0603
- added L7: 8/0.5/2.4, aircoils:SM-L15B
- added OS1: ECS-3225MV-160-CN-TR, IQD-Frequency-Products:3.4X2.7-4-PAD
- added R26: 6k8, rcl:R0805
- added R27: 8k2, rcl:R0805
- added R28: 1k, rcl:R0805
- added R29: 10k, pot:3223W
- added T3: AFT05MS004NT1, AFT05MS004NT1:SOT89-BCE
- added U6: HMC546MS8GETR, HMC546:SOP65P490X110-8N
- LM2: value 22nH -> 16nH
- X1: value 16MHz -> 52746-0871; device IQD-Frequency-Products:HC49 -> con-molex:52745-0890
- moved X1 149.0 mm to (-46.0, -101.9)
Connections:
- removed net N$2: Q1.3, R5.1, T1.1
- removed net N$26: CC3.1, LM2.2
- removed net N$7: R6.2, T1.3
- removed net OSC_OUT: C3.1, U1.13, X1.2
- removed net TFT_LED_A: JP3.15, R6.1
- removed net TRX_RX_SW: U1.5, U2.4
- new net +UB: C46.1, C47.1, C48.2, L7.2
- new net N$15: C27.1, C35.1, L3.2, LM2.2
- new net N$28: R27.2, R29.1
- new net N$33: C_ACG.1, U6.4
- new net N$34: R28.1, R29.3
- new net N$35: C38.1, L4.1, L7.1, T3.D
- new net N$36: C39.1, C40.2, L4.2, L6.1
- new net N$37: C42.1, C43.2, CC3.1, L6.2
- new net N$9: CC3.2, U6.1
- new net PA_BIAS: C37.1, C41.1, C45.2, R26.2
- new net TFT_LED: Q1.3, X1.1
- new net TRX_SW: U1.5, U6.3
- net +3V3: now also OS1.4, R28.2, U6.6, X1.7; no longer C17.1, JP3.2
- net +5V: no longer C11.1, R5.2, T1.2
- net GND: now also C27.2, C35.2, C37.2, C38.2, C39.2, C40.1, C41.2, C42.2, C43.1, C45.1, C46.2, C47.2, C48.1, C_ACG.2, OS1.2, R27.1, T3.S, U6.2, U6.7, X1.8; no longer C1.2, C11.2, C17.2, C3.2, JP3.1, Q2.2, U2.2
- net N$14: no longer Q2.3
- net N$30: now also L3.1, R26.1, T3.G; no longer CC3.2, U2.1
- net N$31: now also U6.5; no longer U2.3
- net N$32: now also U6.8; no longer U2.5
- net OSC_IN: now also OS1.3; no longer C1.1, X1.1
- net SPI1_CS: now also X1.3; no longer JP3.10
- net SPI1_MOSI: now also X1.4; no longer JP3.8
- net SPI1_SCK: now also X1.5; no longer JP3.9
- net SPK_SDN: no longer Q2.1
- net TFT_A0: now also X1.6; no longer JP3.7
- net TFT_RST: now also X1.2; no longer JP3.6
- net TRX_TX_SW: no longer U2.6
Routing:
- net TRX_RX_SW: track 88.8 -> 0.00 mm, vias 2 -> 0
- net TRX_SW: track 0.00 -> 88.7 mm, vias 0 -> 2
- net OSC_OUT: track 16.9 -> 0.00 mm
- net +5V: track 44.2 -> 38.7 mm
- net N$2: track 5.45 -> 0.00 mm
- net N$7: track 3.75 -> 0.00 mm
- net OSC_IN: track 15.6 -> 11.9 mm
- net TFT_LED: track 0.00 -> 3.24 mm
- net TFT_LED_A: track 3.20 -> 0.00 mm
- net GND: track 18.3 -> 16.3 mm, vias 564 -> 562
- net N$26: track 1.91 -> 0.00 mm
- net N$32: track 1.64 -> 0.00 mm
- net N$30: track 1.52 -> 0.00 mm
- net N$14: track 7.31 -> 6.40 mm
- net +3V3: track 360.7 -> 360.1 mm

Commit message: Add files via upload
Parts:
- removed JP1: SWD, pinhead:1X05
- removed X1: 52746-0871, con-molex:52745-0890
- added JP3: SWD, pinhead:1X05/90
- added X4: 52746-0871, con-molex:52745-0890
- C21: device rcl:C1206 -> rcl:C0805
- moved OS1 153.6 mm to (23.2, 37.5)
- moved R2 42.0 mm to (26.6, 37.4), turned to 90 degrees
- moved C_ACG 10.4 mm to (-16.5, 1.91), turned to 90 degrees
- moved C26 3.01 mm to (37.5, 23.2), turned to 270 degrees
- moved C12 2.03 mm to (18.7, 34.9), turned to 90 degrees
- moved L1 1.85 mm to (23.8, 33.3)
- moved C4 0.90 mm to (27.9, 33.7)
- moved C2 0.71 mm to (30.2, 33.7)
Connections:
- net +3V3: now also JP3.5, X4.2; no longer JP1.1, X1.7
- net GND: now also JP3.1, X4.1; no longer JP1.5, X1.8
- net NRST: now also JP3.2; no longer JP1.4
- net SPI1_CS: now also X4.6; no longer X1.3
- net SPI1_MOSI: now also X4.5; no longer X1.4
- net SPI1_SCK: now also X4.4; no longer X1.5
- net SWCLK: now also JP3.3; no longer JP1.3
- net SWDIO: now also JP3.4; no longer JP1.2
- net TFT_A0: now also X4.3; no longer X1.6
- net TFT_LED: now also X4.8; no longer X1.1
- net TFT_RST: now also X4.7; no longer X1.2
Routing:
- net +3V3: track 360.1 -> 0.00 mm, vias 15 -> 0
- net +BATT: track 121.7 -> 0.00 mm, vias 3 -> 0
- net TRX_SW: track 88.7 -> 0.00 mm, vias 2 -> 0
- net SPI1_SCK: track 81.8 -> 0.00 mm, vias 2 -> 0
- net SPI1_MOSI: track 80.3 -> 0.00 mm, vias 2 -> 0
- net ADC2_3: track 79.7 -> 0.00 mm, vias 2 -> 0
- net TRX_TX_SW: track 77.5 -> 0.00 mm, vias 4 -> 0
- net SPI1_CS: track 75.9 -> 0.00 mm, vias 2 -> 0
- net LED_GRN: track 75.2 -> 0.00 mm, vias 2 -> 0
- net LED_RED: track 73.9 -> 0.00 mm, vias 2 -> 0
- net TRX_SDN: track 67.3 -> 0.00 mm, vias 2 -> 0
- net TFT_A0: track 67.1 -> 0.00 mm, vias 2 -> 0
- net TFT_RST: track 66.1 -> 0.00 mm, vias 2 -> 0
- net BLIGHT_CTRL: track 62.1 -> 0.00 mm, vias 2 -> 0
- net SWDIO: track 57.3 -> 0.00 mm, vias 2 -> 0
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
Commit message: Add files via upload
Parts:
- added H1, H2, H3, H4: MOUNT-PAD-ROUND2.8, holes:2,8-PAD
- moved C42 211.7 mm to (39.7, 109.2)
- moved C43 209.0 mm to (34.3, 109.2)
- moved R28 207.9 mm to (25.1, 97.2), turned to 180 degrees
- moved L6 205.7 mm to (36.8, 108.0), turned to 90 degrees
- moved R29 205.3 mm to (26.0, 93.3), turned to 180 degrees
- moved L4 203.2 mm to (36.8, 104.1), turned to 90 degrees
- moved R27 202.8 mm to (28.6, 97.2), turned to 180 degrees
- moved C48 195.8 mm to (29.2, 104.8), turned to 90 degrees
- moved C40 194.1 mm to (39.7, 107.0), turned to 180 degrees
- moved C47 194.0 mm to (31.1, 104.8), turned to 270 degrees
- moved C39 192.3 mm to (39.7, 105.1)
- moved C38 187.4 mm to (36.8, 100.0), turned to 270 degrees
- moved C41 187.2 mm to (29.5, 92.7), turned to 270 degrees
- moved R26 184.3 mm to (32.1, 95.6), turned to 180 degrees
- moved C46 183.2 mm to (31.1, 110.5), turned to 90 degrees
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Connections:
- net GND: now also H1.B2,8, H2.B2,8, H3.B2,8, H4.B2,8
- net PA_BIAS: now also R29.2
Routing:
- net +3V3: track 0.00 -> 29.0 mm, vias 0 -> 3
- net SPK_N: track 0.00 -> 19.9 mm
- net N$27: track 0.00 -> 16.2 mm
- net SPK_P: track 0.00 -> 13.7 mm
- net PA_SUPP: track 0.00 -> 13.3 mm
- net N$13: track 0.00 -> 9.02 mm
- net N$18: track 0.00 -> 8.71 mm
- net N$3: track 0.00 -> 8.65 mm
- net N$17: track 0.00 -> 8.09 mm
- net N$4: track 0.00 -> 7.44 mm
- net N$16: track 0.00 -> 6.36 mm
- net MIC_AMP_IN: track 0.00 -> 6.32 mm
- net ADC1_0: track 0.00 -> 5.92 mm
- net N$14: track 0.00 -> 5.85 mm
- net N$5: track 0.00 -> 4.79 mm
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Other:
- board size 55 x 127 mm -> 42 x 127 mm
- board text added: "TR_9_MAIN_BOARD_1.2"
- board text removed: "TELETRA"
- board text removed: "TR_9_MAIN_BOARD_1.1"
