File: eagle/main.brd (EAGLE design)
At the start: 42 x 127 mm, 127 parts, among them IC1 LD117AS50TR, IC2 LD117AS33TR, IC3 OPA340U, Q1 BSS138, T3 AFT05MS004NT1, U1 STM32F777VIT, U3 L272, U4 ADAM TECH MCSP-Q1-08-A-SG, U5 SI4463-C2A-GM, U6 HMC546MS8GETR, X2 SMA, X3 ILSI 32MHz TCXO, X4 52746-0871

Commit message: Add files via upload
Parts:
- moved X4 91.7 mm to (101.9, 52.7)
- moved R1 78.1 mm to (87.9, 30.2), flipped to the bottom
- moved R21 71.0 mm to (81.9, 27.3), turned to 270 degrees
- moved C24 70.3 mm to (78.1, 22.5)
- moved R22 70.3 mm to (78.1, 30.8)
- moved U$1 70.3 mm to (79.1, 26.7)
- moved JP7 69.9 mm to (89.2, 34.9)
- moved TP2 69.1 mm to (102.2, 37.5)
- moved C16 69.0 mm to (84.8, 50.5)
- moved U4 68.9 mm to (70.2, 40.3)
- moved TP1 68.6 mm to (102.2, 35.2)
- moved C12 68.5 mm to (86.0, 22.2)
- moved C14 68.5 mm to (105.4, 30.2)
- moved C4 68.5 mm to (95.2, 21.0)
- moved L1 68.5 mm to (91.1, 20.6)
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Connections:
- removed net SPK_SDN: U1.1
- removed net TRX_TX_SW: U1.4
Routing:
- net +3V3: track 29.0 -> 234.4 mm, vias 3 -> 9
- net N$31: track 0.00 -> 37.4 mm
- net SPI1_SCK: track 0.00 -> 25.7 mm, vias 0 -> 2
- net SPI1_MOSI: track 0.00 -> 25.2 mm, vias 0 -> 2
- net SPI1_CS: track 0.00 -> 25.2 mm, vias 0 -> 2
- net BLIGHT_CTRL: track 0.00 -> 23.3 mm
- net TFT_RST: track 0.00 -> 21.4 mm
- net TFT_A0: track 0.00 -> 20.1 mm, vias 0 -> 2
- net SD_D0: track 0.00 -> 17.3 mm
- net +BATT: track 2.95 -> 19.9 mm, vias 0 -> 1
- net SD_D1: track 0.00 -> 11.6 mm
- net PA_BIAS: track 0.00 -> 10.7 mm
- net GND: track 0.00 -> 10.3 mm, vias 0 -> 6
- net +5V: track 0.00 -> 9.58 mm
- net VREF: track 0.00 -> 9.31 mm
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
Commit message: Add files via upload
Parts:
- moved JP6 69.0 mm to (23.8, 59.7)
- moved C15 68.9 mm to (22.9, 62.2)
- moved C10 68.7 mm to (9.84, 50.2)
- moved C12 68.7 mm to (17.8, 29.5)
- moved C2 68.7 mm to (28.9, 28.3)
- moved C24 68.7 mm to (9.84, 29.8)
- moved C4 68.7 mm to (27.0, 28.3)
- moved C5 68.7 mm to (36.5, 49.5)
- moved C6 68.7 mm to (18.7, 57.8)
- moved JP7 68.7 mm to (21.0, 42.2)
- moved JP8 68.7 mm to (39.7, 47.3)
- moved L1 68.7 mm to (22.9, 27.9)
- moved Q1 68.7 mm to (37.5, 63.8)
- moved R1 68.7 mm to (19.7, 37.5)
- moved R2 68.7 mm to (25.6, 32.0)
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Connections:
- removed net +UB: C46.1, C47.1, C48.2, L7.2
- net +BATT: now also C46.1, C47.1, C48.2, L7.2
Routing:
- net +3V3: track 234.4 -> 370.9 mm, vias 9 -> 11
- net +BATT: track 19.9 -> 61.4 mm, vias 1 -> 3
- net NRST: track 3.17 -> 38.6 mm, vias 0 -> 1
- net TRX_SDN: track 6.14 -> 41.1 mm
- net TRX_NIRQ: track 4.22 -> 36.6 mm, vias 1 -> 2
- net ADC1_0: track 7.94 -> 37.6 mm, vias 0 -> 2
- net SWCLK: track 0.00 -> 23.9 mm, vias 0 -> 3
- net DAC_OUT: track 0.00 -> 20.7 mm, vias 0 -> 2
- net SWDIO: track 1.29 -> 21.8 mm
- net SPI2_CS: track 1.67 -> 21.7 mm, vias 1 -> 2
- net SPI2_MOSI: track 2.56 -> 20.1 mm, vias 1 -> 2
- net SPI2_MISO: track 2.57 -> 18.7 mm, vias 1 -> 2
- net SPI2_SCK: track 1.68 -> 17.1 mm, vias 1 -> 2
- net GND: track 10.3 -> 20.0 mm, vias 6 -> 16
- net +UB: track 6.56 -> 0.00 mm
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Other:
- board size 42 x 127 mm -> 42.3 x 120 mm

Commit message: Add files via upload
Parts:
- moved H3 16.0 mm to (20.0, 73.0)
Routing:
- net TRX_SW: track 3.92 -> 110.9 mm, vias 2 -> 4
- net +BATT: track 61.4 -> 164.6 mm, vias 3 -> 4
- net LED_RED: track 3.06 -> 88.0 mm, vias 1 -> 2
- net LED_GRN: track 2.16 -> 87.0 mm, vias 1 -> 2
- net ADC2_3: track 6.95 -> 91.5 mm, vias 1 -> 4
- net PTT_INT: track 5.26 -> 58.4 mm, vias 1 -> 3
- net +3V3: track 370.9 -> 358.0 mm
- net GND: track 20.0 -> 23.1 mm, vias 16 -> 160

Commit message: Add files via upload
Routing:
- net +BATT: track 164.6 -> 165.8 mm
- net TFT_A0: track 20.1 -> 19.6 mm
- net GND: vias 160 -> 469

Commit message: Add files via upload
Routing:
- net PTT_INT: vias 3 -> 2
Changed lines of the file:
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@@
 <wire x1="14.605" y1="38.1" x2="14.8675" y2="38.3625" width="0.254" layer="1"/>
 <via x="4.445" y="38.1" extent="1-16" drill="0.2"/>
-<via x="4.445" y="74.295" extent="1-16" drill="0.2"/>
 <wire x1="4.445" y1="38.1" x2="4.445" y2="74.295" width="0.254" layer="1"/>
 <wire x1="4.445" y1="74.295" x2="0.9525" y2="77.7875" width="0.254" layer="1"/>

Commit message: Add files via upload
Routing:
- net GND: vias 469 -> 474
Other:
- board size 42.3 x 120 mm -> 42 x 120 mm
Changed lines of the file:
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@@
 <plain>
 <wire x1="0" y1="0" x2="42" y2="0" width="0" layer="20"/>
-<wire x1="42" y1="0" x2="41.6825" y2="120.015" width="0" layer="20"/>
-<wire x1="41.6825" y1="120.015" x2="-0.3175" y2="120.015" width="0" layer="20"/>
-<wire x1="-0.3175" y1="120.015" x2="0" y2="0" width="0" layer="20"/>
+<wire x1="42" y1="0" x2="42" y2="120" width="0" layer="20"/>
+<wire x1="42" y1="120" x2="0" y2="120" width="0" layer="20"/>
+<wire x1="0" y1="120" x2="0" y2="0" width="0" layer="20"/>
 <text x="12.7" y="20.0025" size="1.778" layer="51" font="vector">TR-9</text>
 <text x="6.6675" y="102.5525" size="1.778" layer="51" font="vector" rot="R270">TR_9_MAIN_BOARD_1.2</text>
@@
 <element name="U1" library="micro-stm_v3" package="LQFP100" value="STM32F777VIT" x="23.8125" y="42.8625"/>
 <element name="U4" library="microsd" package="MICROSD-PUSH-OUT" value="ADAM TECH MCSP-Q1-08-A-SG" x="1.905" y="47.625" rot="R270"/>
-<element name="X2" library="con-coax" package="J502-ND-142-0701-871/876" value="SMA" x="33.7125" y="120.015" rot="R270">
-<attribute name="MPN" value="142-0701-871" x="33.7125" y="120.015" size="1.778" layer="27" rot="R270" display="off"/>
-<attribute name="OC_FARNELL" value="1339835" x="33.7125" y="120.015" size="1.778" layer="27" rot="R270" display="off"/>
-<attribute name="MF" value="JOHNSON COMPONENTS" x="33.7125" y="120.015" size="1.778" layer="27" rot="R270" display="off"/>
-<attribute name="OC_NEWARK" value="91B6105" x="33.7125" y="120.015" size="1.778" layer="27" rot="R270" display="off"/>
+<element name="X2" library="con-coax" package="J502-ND-142-0701-871/876" value="SMA" x="33.7125" y="120" rot="R270">
+<attribute name="MPN" value="142-0701-871" x="33.7125" y="120" size="1.778" layer="27" rot="R270" display="off"/>
+<attribute name="OC_FARNELL" value="1339835" x="33.7125" y="120" size="1.778" layer="27" rot="R270" display="off"/>
+<attribute name="MF" value="JOHNSON COMPONENTS" x="33.7125" y="120" size="1.778" layer="27" rot="R270" display="off"/>
+<attribute name="OC_NEWARK" value="91B6105" x="33.7125" y="120" size="1.778" layer="27" rot="R270" display="off"/>
 </element>
 <element name="U5" library="SI4463-C2A-GM" package="QFN50P400X400X90-20N" value="SI4463-C2A-GM" x="30.7975" y="69.215" rot="R270">
@@
 <via x="11.43" y="1.385" extent="1-16" drill="0.2"/>
 <via x="12.7" y="37.2625" extent="1-16" drill="0.2"/>
+<via x="40.3225" y="82.3475" extent="1-16" drill="0.2"/>
+<via x="38.735" y="79.49" extent="1-16" drill="0.2"/>
+<via x="40.005" y="76.6325" extent="1-16" drill="0.2"/>
+<via x="38.735" y="75.3625" extent="1-16" drill="0.2"/>
+<via x="40.3225" y="73.4575" extent="1-16" drill="0.2"/>
 </signal>
 <signal name="+3V3" class="1">
@@
 <contactref element="X2" pad="1"/>
 <wire x1="33.97" y1="113.9825" x2="33.7125" y2="113.605" width="0.254" layer="1"/>
-<wire x1="33.7125" y1="113.605" x2="33.7125" y2="117.4496" width="0.5" layer="1"/>
+<wire x1="33.7125" y1="113.605" x2="33.7125" y2="117.4346" width="0.5" layer="1"/>
 <wire x1="33.97" y1="113.9825" x2="35.88" y2="113.9825" width="0.254" layer="1"/>
 </signal>
