File: eagle/main.sch (EAGLE design)
At the start: 81 parts, among them IC1 LD117AS50TR, IC2 LD117AS33TR, IC3 OPA340U, Q1 BSS138, T1 FDV304P, U1 STM32F777VIT, U2 RFM26W, U3 PAM8302, U4 MICROSD-PUSH-OUT, X1 16MHz, X2 SMA

Commit message: Add files via upload
Parts:
- R5: value 47k -> 1k
Changed lines of the file:
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@@
 <part name="JP3" library="pinhead" deviceset="PINHD-1X16" device="" value="TFT_CONN"/>
 <part name="Q1" library="bss138_10" deviceset="BSS138" device=""/>
-<part name="R5" library="rcl" deviceset="R-EU_" device="R0805" value="47k"/>
+<part name="R5" library="rcl" deviceset="R-EU_" device="R0805" value="1k"/>
 <part name="R6" library="rcl" deviceset="R-EU_" device="R1206" value="22R"/>
 <part name="GND23" library="supply1" deviceset="GND" device=""/>

Commit message: Add files via upload
Connections:
- net ADC1_0: now also R7.2; no longer R7.1, R8.2
- net N$4: now also R7.1, R8.2; no longer R7.2
Other:
- moved on the sheet: R7
Changed lines of the file:
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@@
 <instance part="JP5" gate="G$1" x="162.56" y="154.94" rot="R90"/>
 <instance part="GND37" gate="1" x="162.56" y="144.78"/>
-<instance part="R7" gate="G$1" x="55.88" y="132.08" rot="R90"/>
+<instance part="R7" gate="G$1" x="43.18" y="121.92" rot="R180"/>
 <instance part="R8" gate="G$1" x="55.88" y="114.3" rot="R90"/>
 <instance part="GND26" gate="1" x="48.26" y="129.54"/>
@@
 <wire x1="38.1" y1="139.7" x2="30.48" y2="139.7" width="0.1524" layer="91"/>
 <wire x1="30.48" y1="139.7" x2="30.48" y2="121.92" width="0.1524" layer="91"/>
-<pinref part="R7" gate="G$1" pin="1"/>
-<wire x1="30.48" y1="121.92" x2="55.88" y2="121.92" width="0.1524" layer="91"/>
-<pinref part="R8" gate="G$1" pin="2"/>
-<wire x1="55.88" y1="127" x2="55.88" y2="121.92" width="0.1524" layer="91"/>
-<junction x="55.88" y="121.92"/>
-<wire x1="55.88" y1="121.92" x2="55.88" y2="119.38" width="0.1524" layer="91"/>
 <wire x1="30.48" y1="139.7" x2="27.94" y2="139.7" width="0.1524" layer="91"/>
 <label x="27.94" y="139.7" size="1.27" layer="95" rot="R180" xref="yes"/>
 <junction x="30.48" y="139.7"/>
-</segment>
-</net>
-<net name="N$4" class="0">
-<segment>
 <pinref part="R7" gate="G$1" pin="2"/>
-<pinref part="IC3" gate="G$1" pin="-IN"/>
-<wire x1="55.88" y1="137.16" x2="53.34" y2="137.16" width="0.1524" layer="91"/>
+<wire x1="30.48" y1="121.92" x2="38.1" y2="121.92" width="0.1524" layer="91"/>
 </segment>
 </net>
@@
 </segment>
 </net>
+<net name="N$4" class="0">
+<segment>
+<pinref part="R8" gate="G$1" pin="2"/>
+<wire x1="55.88" y1="121.92" x2="55.88" y2="119.38" width="0.1524" layer="91"/>
+<pinref part="R7" gate="G$1" pin="1"/>
+<wire x1="48.26" y1="121.92" x2="55.88" y2="121.92" width="0.1524" layer="91"/>
+<wire x1="55.88" y1="121.92" x2="55.88" y2="137.16" width="0.1524" layer="91"/>
+<pinref part="IC3" gate="G$1" pin="-IN"/>
+<wire x1="55.88" y1="137.16" x2="53.34" y2="137.16" width="0.1524" layer="91"/>
+<junction x="55.88" y="121.92"/>
+</segment>
+</net>

Commit message: Add files via upload
Parts:
- added C0: 8p2, rcl:C-EUC0805
- added C34: 10n, rcl:C-EUC0805
- added CC1, CC2, CC3: 1000p, rcl:C-EUC0805
- added CM: 13p, rcl:C-EUC0805
- added CM1, CM2, CM3: 9p1, rcl:C-EUC0805
- added CR1: 3p9, rcl:C-EUC0805
- added CR2: 2p2, rcl:C-EUC0805
- added L0: 30nH, resistor:R-EU_R0805
- added LCHOKE: 220nH, resistor:R-EU_R0805
- added LM1: 27nH, resistor:R-EU_R0805
- added LM2: 22nH, resistor:R-EU_R0805
- added LM3: 15nH, resistor:R-EU_R0805
- added LR1: 56nH, resistor:R-EU_R0805
- added LR2: 51nH, resistor:R-EU_R0805
- added U5: SI4463-C2A-GM, SI4463-C2A-GM:SI4463-C2A-GM
- added X3: ILSI 32MHz TCXO, ILSI_tcxo:ASE
- U2: value RFM26W -> CG2179M2; device hoperf:RFM26W -> CG2179M2:CG2179M2
Connections:
- removed net N$3: U2.ANT, X2.1
- new net 32M: U5.XIN, X3.OUT
- new net N$21: CM3.1, LM3.2, X2.1
- new net N$22: CC2.2, CM2.1, LM3.1
- new net N$23: C0.2, L0.1
- new net N$24: CM.1, L0.2, LM1.1
- new net N$25: CM1.1, LM1.2, LM2.1
- new net N$26: CC3.1, LM2.2
- new net N$29: CC1.1, CR2.2, LR2.2
- new net N$30: CC3.2, U2.RF1
- new net N$31: CC1.2, U2.RF2
- new net N$32: CC2.1, U2.RFC
- new net RXN: CR1.1, LR1.1, LR2.1, U5.RXN
- new net RXP: CR2.1, LR1.2, U5.RXP
- new net TX: C0.1, LCHOKE.1, U5.TX
- net +3V3: now also C34.1, LCHOKE.2, U5.VDD, X3.VDD; no longer U2.VCC
- net GND: now also C34.2, CM.2, CM1.2, CM2.2, CM3.2, CR1.2, U2.GND, U5.GND, X3.GND; no longer U2.GND@1, U2.GND@2
- net SPI1_CS: now also U5.NSEL; no longer U2.NSEL
- net SPI1_MISO: now also U5.SDO; no longer U2.SDO
- net SPI1_MOSI: now also U5.SDI; no longer U2.SDI
- net SPI1_SCK: now also U5.SCLK; no longer U2.SCK
- net TRX_NIRQ: now also U5.NIRQ; no longer U2.NIRQ
- net TRX_RX_SW: no longer U2.RX-ANT
- net TRX_SDN: now also U5.SDN; no longer U2.SDN
- net TRX_TX_SW: no longer U2.TX-ANT
Other:
- moved on the sheet: X2

Commit message: Add files via upload
Parts:
- removed C24, C25, C27: 220p, rcl:C-EUC1206
- removed L3, L4: (no value), inductor-neosid:SM-B5
- removed U3: PAM8302, pam:PAM8302
- added IC4: L272D, linear:L272D
- added Q2: BSS138, bss138_10:BSS138
- added R19, R20, R23, R24: 10k, resistor:R-EU_R0805
- added R21, R22, R25: 22k, resistor:R-EU_R0805
- R13, R14: value 10k -> 4k7
- R7: value 680R -> 820R
Connections:
- removed net +UB: C8.+, IC1.IN, JP2.2, R3.2
- removed net SPK_INT_N: C25.1, JP4.2, L4.2
- removed net SPK_INT_P: C24.2, JP4.1, L3.2
- new net +BATT: C32.1, C8.+, IC1.IN, JP2.2, L5.1, R14.1, R3.2
- new net N$27: IC4B.+IN, R22.2
- new net N$28: IC4B.-IN, R23.2, R24.1
- new net N$3: IC4A.-IN, R19.1, R20.2
- new net N$33: IC4B.OUT, JP4.1, R24.2
- net +5V: no longer C32.1, L5.1
- net GND: now also C30.1, IC4P.GND, Q2.S, R13.2; no longer C24.1, C25.2, C27.2, C30.2, R14.1, U3.GND
- net N$13: now also C30.2, R13.1, R14.2, R21.1, R22.1, R25.1; no longer L4.1, U3.VO-
- net N$14: now also Q2.D, R19.2, R25.2; no longer C27.1, U3.IN+
- net N$15: now also IC4A.+IN, R21.2; no longer C30.1, R13.1, R14.2, U3.IN-
- net N$8: now also IC4P.V+; no longer R13.2, U3.VDD
- net N$9: now also IC4A.OUT, JP4.2, R20.1, R23.1; no longer L3.1, U3.VO+
- net SPK_SDN: now also Q2.G; no longer U3./SD
Other:
- moved on the sheet: C26, C29, C30, C31, C32, JP4, L5, R13, R14

Commit message: Add files via upload
Parts:
- removed IC4: L272D, linear:L272D
- removed R21, R22: 22k, resistor:R-EU_R0805
- added U3: L272, L272:L272
- C26: value 1u -> 470n
- R20: value 10k -> 15k
Connections:
- removed net N$15: IC4A.+IN, R21.2
- removed net N$28: IC4B.-IN, R23.2, R24.1
- removed net N$33: IC4B.OUT, JP4.1, R24.2
- removed net N$8: C29.1, C31.1, IC4P.V+, L5.2
- removed net N$9: IC4A.OUT, JP4.2, R20.1, R23.1
- new net PA_SUPP: C29.1, C31.1, L5.2, U3.SUPP
- new net SPK_N: JP4.2, R20.2, R24.2, U3.OUT1
- new net SPK_P: JP4.1, R23.2, U3.OUT2
- net GND: now also U3.GND; no longer IC4P.GND
- net N$13: now also R23.1, R24.1, U3.IN2-; no longer C30.2, R13.1, R14.2, R21.1, R22.1, R25.1
- net N$27: now also C30.2, R13.1, R14.2, R25.1, U3.IN1+, U3.IN2+; no longer IC4B.+IN, R22.2
- net N$3: now also R20.1, U3.IN1-; no longer IC4A.-IN, R20.2
Other:
- moved on the sheet: C29, C31, C32, JP4, L5, R14, R20, R23, R24, R25

Commit message: Add files via upload
Parts:
- removed JP9: ACC_CONN, pinhead:PINHD-1X4
- added U$1: ADXL345, adxl345:ADXL345
Connections:
- net +3V3: now also U$1.!CS, U$1.VDDIO; no longer JP9.1
- net GND: now also U$1.GND$1, U$1.GND$2, U$1.GND$3, U$1.MISO, U$1.VS; no longer JP9.4
- net I2C1_SCL: now also U$1.SCLK; no longer JP9.2
- net I2C1_SDA: now also U$1.MOSI; no longer JP9.3
Other:
- note added: "ADDR 0x53"
- note added: "ALT ADDRESS"
- note added: "SCL"
- note added: "SDA"

Commit message: Add files via upload
Parts:
- added D1: CGRM4007-G, diode:CGRM4007-G
- added U$2: 2A, chiptron_cz:SMD-FUSE
- C10, C12, C13, C14, C15, C16, C17, C18: device resistor:CPOL-EUSMCC -> resistor:C-EUC1206
- JP2: device pinhead:PINHD-1X2 -> pinhead:PINHD-1X3/90
- U4: value MICROSD-PUSH-OUT -> ADAM TECH MCSP-Q1-08-A-SG
Connections:
- new net N$8: JP2.3, U$2.P$1
- net +3V3: now also C10.1, C12.1, C13.1, C14.1, C15.1, C16.1, C17.1, C18.1; no longer C10.+, C12.+, C13.+, C14.+, C15.+, C16.+, C17.+, C18.+
- net +BATT: now also D1.C; no longer JP2.2
- net GND: now also C10.2, C12.2, C13.2, C14.2, C15.2, C16.2, C17.2, C18.2, D1.A; no longer C10.-, C12.-, C13.-, C14.-, C15.-, C16.-, C17.-, C18.-
- net SPI1_CS: now also JP3.10; no longer U5.NSEL
- net SPI1_MISO: no longer U5.SDO
- net SPI1_MOSI: now also JP3.8; no longer U5.SDI
- net SPI1_SCK: now also JP3.9; no longer U5.SCLK
- net SPI2_CS: now also U5.NSEL; no longer JP3.10
- net SPI2_MISO: now also U5.SDO
- net SPI2_MOSI: now also U5.SDI; no longer JP3.8
- net SPI2_SCK: now also U5.SCLK; no longer JP3.9

Commit message: Add files via upload
Parts:
- added R21, R22: 4k7, rcl:R-EU_R0805
Connections:
- net +3V3: now also R21.2, R22.2
- net +BATT: now also U$2.P$2
- net GND: now also JP2.3; no longer JP2.1
- net I2C1_SCL: now also R22.1
- net I2C1_SDA: now also R21.1
- net N$8: now also JP2.1; no longer JP2.3
Other:
- moved on the sheet: JP2, U$1
Changed lines of the file:
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@@
 <part name="GND43" library="supply1" deviceset="GND" device=""/>
 <part name="D1" library="diode" deviceset="CGRM400*-G" device="" technology="7"/>
+<part name="R21" library="rcl" deviceset="R-EU_" device="R0805" value="4k7"/>
+<part name="R22" library="rcl" deviceset="R-EU_" device="R0805" value="4k7"/>
+<part name="+3V6" library="supply1" deviceset="+3V3" device=""/>
+<part name="+3V7" library="supply1" deviceset="+3V3" device=""/>
 </parts>
 <sheets>
@@
 <instance part="GND16" gate="1" x="58.42" y="96.52"/>
 <instance part="C9" gate="G$1" x="91.44" y="96.52"/>
-<instance part="JP2" gate="A" x="45.72" y="137.16" rot="R180"/>
+<instance part="JP2" gate="A" x="45.72" y="137.16" rot="MR0"/>
 <instance part="SUPPLY1" gate="G$1" x="66.04" y="144.78"/>
 <instance part="GND15" gate="1" x="53.34" y="127"/>
@@
 </segment>
 <segment>
-<pinref part="JP2" gate="A" pin="1"/>
 <pinref part="GND15" gate="1" pin="GND"/>
-<wire x1="48.26" y1="134.62" x2="53.34" y2="134.62" width="0.1524" layer="91"/>
 <wire x1="53.34" y1="134.62" x2="53.34" y2="129.54" width="0.1524" layer="91"/>
+<pinref part="JP2" gate="A" pin="3"/>
+<wire x1="53.34" y1="134.62" x2="48.26" y2="134.62" width="0.1524" layer="91"/>
 </segment>
 <segment>
@@
 <segment>
 <pinref part="SUPPLY1" gate="G$1" pin="+UB"/>
-<wire x1="63.5" y1="139.7" x2="66.04" y2="139.7" width="0.1524" layer="91"/>
-<wire x1="66.04" y1="139.7" x2="66.04" y2="142.24" width="0.1524" layer="91"/>
 <pinref part="D1" gate="G$1" pin="C"/>
 <wire x1="66.04" y1="137.16" x2="66.04" y2="139.7" width="0.1524" layer="91"/>
+<pinref part="U$2" gate="G$1" pin="P$2"/>
+<wire x1="66.04" y1="139.7" x2="66.04" y2="142.24" width="0.1524" layer="91"/>
+<wire x1="63.5" y1="139.7" x2="66.04" y2="139.7" width="0.1524" layer="91"/>
 <junction x="66.04" y="139.7"/>
 </segment>
@@
 <segment>
 <pinref part="U$2" gate="G$1" pin="P$1"/>
-<pinref part="JP2" gate="A" pin="3"/>
+<pinref part="JP2" gate="A" pin="1"/>
 <wire x1="53.34" y1="139.7" x2="48.26" y2="139.7" width="0.1524" layer="91"/>
 </segment>
@@
 <sheet>
 <plain>
-<text x="167.64" y="106.68" size="1.27" layer="91">ALT ADDRESS</text>
-<text x="167.64" y="111.76" size="1.27" layer="91">SDA</text>
-<text x="167.64" y="101.6" size="1.27" layer="91">SCL</text>
-<text x="137.16" y="121.92" size="1.27" layer="91">ADDR 0x53</text>
+<text x="162.56" y="106.68" size="2.54" layer="97">ALT ADDRESS</text>
+<text x="162.56" y="111.76" size="2.54" layer="97">SDA</text>
+<text x="162.56" y="101.6" size="2.54" layer="97">SCL</text>
+<text x="104.14" y="66.04" size="2.54" layer="97">ADDR 0x53</text>
 </plain>
 <instances>
-<instance part="GND33" gate="1" x="106.68" y="86.36"/>
-<instance part="+3V4" gate="G$1" x="106.68" y="119.38"/>
+<instance part="GND33" gate="1" x="91.44" y="86.36"/>
+<instance part="+3V4" gate="G$1" x="91.44" y="119.38"/>
 <instance part="FRAME7" gate="G$1" x="0" y="0"/>
-<instance part="U$1" gate="G$1" x="127" y="93.98"/>
-<instance part="+3V5" gate="G$1" x="149.86" y="96.52" rot="R270"/>
-<instance part="GND36" gate="1" x="149.86" y="106.68" rot="R90"/>
+<instance part="U$1" gate="G$1" x="111.76" y="93.98"/>
+<instance part="+3V5" gate="G$1" x="134.62" y="96.52" rot="R270"/>
+<instance part="GND36" gate="1" x="134.62" y="106.68" rot="R90"/>
+<instance part="R21" gate="G$1" x="137.16" y="119.38" rot="R90"/>
+<instance part="R22" gate="G$1" x="144.78" y="119.38" rot="R90"/>
+<instance part="+3V6" gate="G$1" x="137.16" y="129.54"/>
+<instance part="+3V7" gate="G$1" x="144.78" y="129.54"/>
 </instances>
 <busses>
@@
 <net name="I2C1_SCL" class="0">
 <segment>
-<wire x1="149.86" y1="101.6" x2="142.24" y2="101.6" width="0.1524" layer="91"/>
-<label x="149.86" y="101.6" size="1.27" layer="95" xref="yes"/>
+<wire x1="147.32" y1="101.6" x2="144.78" y2="101.6" width="0.1524" layer="91"/>
+<label x="147.32" y="101.6" size="1.27" layer="95" xref="yes"/>
 <pinref part="U$1" gate="G$1" pin="SCLK"/>
+<pinref part="R22" gate="G$1" pin="1"/>
+<wire x1="144.78" y1="101.6" x2="127" y2="101.6" width="0.1524" layer="91"/>
+<wire x1="144.78" y1="114.3" x2="144.78" y2="101.6" width="0.1524" layer="91"/>
+<junction x="144.78" y="101.6"/>
 </segment>
 </net>
 <net name="I2C1_SDA" class="0">
 <segment>
-<wire x1="149.86" y1="111.76" x2="142.24" y2="111.76" width="0.1524" layer="91"/>
-<label x="149.86" y="111.76" size="1.27" layer="95" xref="yes"/>
+<wire x1="147.32" y1="111.76" x2="137.16" y2="111.76" width="0.1524" layer="91"/>
+<label x="147.32" y="111.76" size="1.27" layer="95" xref="yes"/>
 <pinref part="U$1" gate="G$1" pin="MOSI"/>
+<pinref part="R21" gate="G$1" pin="1"/>
+<wire x1="137.16" y1="111.76" x2="127" y2="111.76" width="0.1524" layer="91"/>
+<wire x1="137.16" y1="114.3" x2="137.16" y2="111.76" width="0.1524" layer="91"/>
+<junction x="137.16" y="111.76"/>
 </segment>
 </net>
@@
 <pinref part="U$1" gate="G$1" pin="VDDIO"/>
 <pinref part="+3V4" gate="G$1" pin="+3V3"/>
-<wire x1="111.76" y1="111.76" x2="106.68" y2="111.76" width="0.1524" layer="91"/>
-<wire x1="106.68" y1="111.76" x2="106.68" y2="116.84" width="0.1524" layer="91"/>
+<wire x1="96.52" y1="111.76" x2="91.44" y2="111.76" width="0.1524" layer="91"/>
+<wire x1="91.44" y1="111.76" x2="91.44" y2="116.84" width="0.1524" layer="91"/>
 </segment>
 <segment>
 <pinref part="+3V5" gate="G$1" pin="+3V3"/>
 <pinref part="U$1" gate="G$1" pin="!CS"/>
-<wire x1="147.32" y1="96.52" x2="142.24" y2="96.52" width="0.1524" layer="91"/>
+<wire x1="132.08" y1="96.52" x2="127" y2="96.52" width="0.1524" layer="91"/>
+</segment>
+<segment>
+<pinref part="R21" gate="G$1" pin="2"/>
+<pinref part="+3V6" gate="G$1" pin="+3V3"/>
+<wire x1="137.16" y1="127" x2="137.16" y2="124.46" width="0.1524" layer="91"/>
+</segment>
+<segment>
+<pinref part="R22" gate="G$1" pin="2"/>
+<pinref part="+3V7" gate="G$1" pin="+3V3"/>
+<wire x1="144.78" y1="127" x2="144.78" y2="124.46" width="0.1524" layer="91"/>
 </segment>
 </net>
@@
 <pinref part="U$1" gate="G$1" pin="VS"/>
 <pinref part="GND33" gate="1" pin="GND"/>
-<wire x1="111.76" y1="106.68" x2="106.68" y2="106.68" width="0.1524" layer="91"/>
-<wire x1="106.68" y1="106.68" x2="106.68" y2="101.6" width="0.1524" layer="91"/>
-<wire x1="106.68" y1="88.9" x2="106.68" y2="91.44" width="0.1524" layer="91"/>
+<wire x1="96.52" y1="106.68" x2="91.44" y2="106.68" width="0.1524" layer="91"/>
+<wire x1="91.44" y1="106.68" x2="91.44" y2="101.6" width="0.1524" layer="91"/>
+<wire x1="91.44" y1="88.9" x2="91.44" y2="91.44" width="0.1524" layer="91"/>
 <pinref part="U$1" gate="G$1" pin="GND$3"/>
-<wire x1="111.76" y1="91.44" x2="106.68" y2="91.44" width="0.1524" layer="91"/>
-<wire x1="106.68" y1="91.44" x2="106.68" y2="96.52" width="0.1524" layer="91"/>
+<wire x1="96.52" y1="91.44" x2="91.44" y2="91.44" width="0.1524" layer="91"/>
+<wire x1="91.44" y1="91.44" x2="91.44" y2="96.52" width="0.1524" layer="91"/>
 <pinref part="U$1" gate="G$1" pin="GND$2"/>
-<wire x1="111.76" y1="96.52" x2="106.68" y2="96.52" width="0.1524" layer="91"/>
-<wire x1="106.68" y1="96.52" x2="106.68" y2="101.6" width="0.1524" layer="91"/>
+<wire x1="96.52" y1="96.52" x2="91.44" y2="96.52" width="0.1524" layer="91"/>
+<wire x1="91.44" y1="96.52" x2="91.44" y2="101.6" width="0.1524" layer="91"/>
 <pinref part="U$1" gate="G$1" pin="GND$1"/>
-<wire x1="106.68" y1="101.6" x2="111.76" y2="101.6" width="0.1524" layer="91"/>
-<junction x="106.68" y="101.6"/>
-<junction x="106.68" y="96.52"/>
-<junction x="106.68" y="91.44"/>
+<wire x1="91.44" y1="101.6" x2="96.52" y2="101.6" width="0.1524" layer="91"/>
+<junction x="91.44" y="101.6"/>
+<junction x="91.44" y="96.52"/>
+<junction x="91.44" y="91.44"/>
 </segment>
 <segment>
 <pinref part="GND36" gate="1" pin="GND"/>
 <pinref part="U$1" gate="G$1" pin="MISO"/>
-<wire x1="147.32" y1="106.68" x2="142.24" y2="106.68" width="0.1524" layer="91"/>
-</segment>
-</net>
+<wire x1="132.08" y1="106.68" x2="127" y2="106.68" width="0.1524" layer="91"/>
+</segment>
+</net>
