File: eagle/main.sch (EAGLE design)
At the start: 106 parts, among them IC1 LD117AS50TR, IC2 LD117AS33TR, IC3 OPA340U, Q1 BSS138, Q2 BSS138, T1 FDV304P, U1 STM32F777VIT, U2 CG2179M2, U3 L272, U4 ADAM TECH MCSP-Q1-08-A-SG, U5 SI4463-C2A-GM, X1 16MHz, X2 SMA, X3 ILSI 32MHz TCXO

Commit message: Add files via upload
Parts:
- added C24, C25: 10n, resistor:C-EUC0805
- C26, C32: device rcl:C-EUC1206 -> rcl:C-EUC0805
Connections:
- net +3V3: now also C24.1, C25.1
- net GND: now also C24.2, C25.2
- net TRX_RX_SW: now also U2.VC2
- net TRX_TX_SW: now also U2.VC1
Other:
- note added: "SD, RFM, GPS, TFT, OPA, ACCEL"
- note removed: "SD, RFM, GPS, TFT, OPA"

Commit message: Add files via upload
Connections:
- net +3V3: now also U$1.VS
- net GND: no longer U$1.VS
Changed lines of the file:
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@@
 <wire x1="96.52" y1="111.76" x2="91.44" y2="111.76" width="0.1524" layer="91"/>
 <wire x1="91.44" y1="111.76" x2="91.44" y2="116.84" width="0.1524" layer="91"/>
+<pinref part="U$1" gate="G$1" pin="VS"/>
+<wire x1="96.52" y1="106.68" x2="91.44" y2="106.68" width="0.1524" layer="91"/>
+<wire x1="91.44" y1="106.68" x2="91.44" y2="111.76" width="0.1524" layer="91"/>
+<junction x="91.44" y="111.76"/>
 </segment>
 <segment>
@@
 <net name="GND" class="1">
 <segment>
-<pinref part="U$1" gate="G$1" pin="VS"/>
 <pinref part="GND33" gate="1" pin="GND"/>
-<wire x1="96.52" y1="106.68" x2="91.44" y2="106.68" width="0.1524" layer="91"/>
-<wire x1="91.44" y1="106.68" x2="91.44" y2="101.6" width="0.1524" layer="91"/>
 <wire x1="91.44" y1="88.9" x2="91.44" y2="91.44" width="0.1524" layer="91"/>
 <pinref part="U$1" gate="G$1" pin="GND$3"/>
@@
 <pinref part="U$1" gate="G$1" pin="GND$1"/>
 <wire x1="91.44" y1="101.6" x2="96.52" y2="101.6" width="0.1524" layer="91"/>
-<junction x="91.44" y="101.6"/>
 <junction x="91.44" y="96.52"/>
 <junction x="91.44" y="91.44"/>

Commit message: Add files via upload
Parts:
- removed C1, C3: 18p, rcl:C-EUC0805
- removed C11: 10u, resistor:C-EUC1206
- removed C17: 22u/TA, resistor:C-EUC1206
- removed JP3: TFT_CONN, pinhead:PINHD-1X16
- removed Q2: BSS138, bss138_10:BSS138
- removed R5: 1k, rcl:R-EU_R0805
- removed R6: 22R, rcl:R-EU_R1206
- removed T1: FDV304P, FDV304P:FDV304P
- removed U2: CG2179M2, CG2179M2:CG2179M2
- added C27, C35, C38, C42: 10p, rcl:C-EUC0805
- added C37, C47: 100p, rcl:C-EUC0805
- added C39: 12p, rcl:C-EUC0805
- added C40: 7p, rcl:C-EUC0805
- added C41, C48: 1000p, rcl:C-EUC0805
- added C43: 2p, rcl:C-EUC0805
- added C45, C46: 1u/TA, resistor:C-EUC1206
- added C_ACG: 33p, rcl:C-EUC0805
- added L3: 2.7nH, rcl:R-EU_R0805
- added L4, L6: 1nH, resistor:R-EU_R0603
- added L7: 8/0.5/2.4, aircoils:AIR_COIL
- added OS1: ECS-3225MV-160-CN-TR, IQD-Frequency-Products:OSC-OE-CFPS-39
- added R26: 6k8, rcl:R-EU_R0805
- added R27: 8k2, rcl:R-EU_R0805
- added R28: 1k, rcl:R-EU_R0805
- added R29: 10k, pot:TRIM_EU-3223W
- added T3: AFT05MS004NT1, AFT05MS004NT1:AFT05MS004NT1
- added U6: HMC546MS8GETR, HMC546:HMC546MS8GETR
- LM2: value 22nH -> 16nH
- X1: value 16MHz -> 52746-0871; device IQD-Frequency-Products:CRYSTALS-NOGND-HC49 -> con-molex:52745-0890
Connections:
- removed net N$2: Q1.D, R5.1, T1.G
- removed net N$26: CC3.1, LM2.2
- removed net N$7: R6.2, T1.D
- removed net OSC_OUT: C3.1, U1.P$13, X1.2
- removed net TFT_LED_A: JP3.15, R6.1
- removed net TRX_RX_SW: U1.P$5, U2.VC2
- new net +UB: C46.1, C47.1, C48.2, L7.2
- new net N$15: C27.1, C35.1, L3.2, LM2.2
- new net N$28: R27.2, R29.A
- new net N$33: C_ACG.1, U6.ACG
- new net N$34: R28.1, R29.E
- new net N$35: C38.1, L4.1, L7.1, T3.D
- new net N$36: C39.1, C40.2, L4.2, L6.1
- new net N$37: C42.1, C43.2, CC3.1, L6.2
- new net N$9: CC3.2, U6.TX
- new net PA_BIAS: C37.1, C41.1, C45.2, R26.2
- new net TFT_LED: Q1.D, X1-1.S
- new net TRX_SW: U1.P$5, U6.VCTL
- net +3V3: now also OS1.VDD, R28.2, U6.VDD, X1-7.S; no longer C17.1, JP3.2
- net +5V: no longer C11.1, R5.2, T1.S
- net GND: now also C27.2, C35.2, C37.2, C38.2, C39.2, C40.1, C41.2, C42.2, C43.1, C45.1, C46.2, C47.2, C48.1, C_ACG.2, OS1.VSS, R27.1, T3.S, U6.GND1, U6.GND2, X1-8.S; no longer C1.2, C11.2, C17.2, C3.2, JP3.1, Q2.S, U2.GND
- net N$14: no longer Q2.D
- net N$30: now also L3.1, R26.1, T3.G; no longer CC3.2, U2.RF1
- net N$31: now also U6.RX; no longer U2.RF2
- net N$32: now also U6.RFC; no longer U2.RFC
- net OSC_IN: now also OS1.OUT; no longer C1.1, X1.1
- net SPI1_CS: now also X1-3.S; no longer JP3.10
- net SPI1_MOSI: now also X1-4.S; no longer JP3.8
- net SPI1_SCK: now also X1-5.S; no longer JP3.9
- net SPK_SDN: no longer Q2.G
- net TFT_A0: now also X1-6.S; no longer JP3.7
- net TFT_RST: now also X1-2.S; no longer JP3.6
- net TRX_TX_SW: no longer U2.VC1
Other:
- note added: "SD, RFM, GPS, OPA, ACCEL"
- note removed: "BACKLIGHT"
- note removed: "SD, RFM, GPS, TFT, OPA, ACCEL"

Commit message: Add files via upload
Parts:
- removed JP1: SWD, pinhead:PINHD-1X5
- removed X1: 52746-0871, con-molex:52745-0890
- added JP3: SWD, pinhead:PINHD-1X5/90
- added X4: 52746-0871, con-molex:52745-0890
- C21: device rcl:C-EUC1206 -> rcl:C-EUC0805
Connections:
- net +3V3: now also JP3.5, X4-2.S; no longer JP1.1, X1-7.S
- net GND: now also JP3.1, X4-1.S; no longer JP1.5, X1-8.S
- net NRST: now also JP3.2; no longer JP1.4
- net SPI1_CS: now also X4-6.S; no longer X1-3.S
- net SPI1_MOSI: now also X4-5.S; no longer X1-4.S
- net SPI1_SCK: now also X4-4.S; no longer X1-5.S
- net SWCLK: now also JP3.3; no longer JP1.3
- net SWDIO: now also JP3.4; no longer JP1.2
- net TFT_A0: now also X4-3.S; no longer X1-6.S
- net TFT_LED: now also X4-8.S; no longer X1-1.S
- net TFT_RST: now also X4-7.S; no longer X1-2.S

Commit message: Add files via upload
Parts:
- added H1, H2, H3, H4: MOUNT-PAD-ROUND2.8, holes:MOUNT-PAD-ROUND2.8
Connections:
- net GND: now also H1.MOUNT, H2.MOUNT, H3.MOUNT, H4.MOUNT
- net PA_BIAS: now also R29.S
Changed lines of the file:
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@@
 <part name="JP3" library="pinhead" deviceset="PINHD-1X5" device="/90" value="SWD"/>
 <part name="X4" library="con-molex" deviceset="52745-0890" device="" value="52746-0871"/>
+<part name="H1" library="holes" deviceset="MOUNT-PAD-ROUND" device="2.8"/>
+<part name="H2" library="holes" deviceset="MOUNT-PAD-ROUND" device="2.8"/>
+<part name="H3" library="holes" deviceset="MOUNT-PAD-ROUND" device="2.8"/>
+<part name="H4" library="holes" deviceset="MOUNT-PAD-ROUND" device="2.8"/>
+<part name="GND1" library="supply1" deviceset="GND" device=""/>
+<part name="GND22" library="supply1" deviceset="GND" device=""/>
+<part name="GND29" library="supply1" deviceset="GND" device=""/>
+<part name="GND63" library="supply1" deviceset="GND" device=""/>
 </parts>
 <sheets>
@@
 <instance part="C24" gate="G$1" x="195.58" y="91.44"/>
 <instance part="C25" gate="G$1" x="205.74" y="91.44"/>
+<instance part="H1" gate="G$1" x="38.1" y="30.48" rot="R90"/>
+<instance part="H2" gate="G$1" x="45.72" y="30.48" rot="R90"/>
+<instance part="H3" gate="G$1" x="53.34" y="30.48" rot="R90"/>
+<instance part="H4" gate="G$1" x="60.96" y="30.48" rot="R90"/>
+<instance part="GND1" gate="1" x="38.1" y="25.4"/>
+<instance part="GND22" gate="1" x="45.72" y="25.4"/>
+<instance part="GND29" gate="1" x="53.34" y="25.4"/>
+<instance part="GND63" gate="1" x="60.96" y="25.4"/>
 </instances>
 <busses>
@@
 <pinref part="D1" gate="G$1" pin="A"/>
 <wire x1="66.04" y1="129.54" x2="66.04" y2="132.08" width="0.1524" layer="91"/>
+</segment>
+<segment>
+<pinref part="H1" gate="G$1" pin="MOUNT"/>
+<pinref part="GND1" gate="1" pin="GND"/>
+</segment>
+<segment>
+<pinref part="H2" gate="G$1" pin="MOUNT"/>
+<pinref part="GND22" gate="1" pin="GND"/>
+</segment>
+<segment>
+<pinref part="H3" gate="G$1" pin="MOUNT"/>
+<pinref part="GND29" gate="1" pin="GND"/>
+</segment>
+<segment>
+<pinref part="H4" gate="G$1" pin="MOUNT"/>
+<pinref part="GND63" gate="1" pin="GND"/>
 </segment>
 </net>
@@
 <wire x1="220.98" y1="144.78" x2="215.9" y2="144.78" width="0.1524" layer="91"/>
 <label x="215.9" y="144.78" size="1.778" layer="95" rot="R180" xref="yes"/>
-</segment>
-</net>
+<pinref part="R29" gate="1" pin="S"/>
+</segment>
+</net>

Commit message: Add files via upload
Connections:
- removed net SPK_SDN: U1.P$1
- removed net TRX_TX_SW: U1.P$4
Changed lines of the file:
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@@
-</segment>
-</net>
-<net name="SPK_SDN" class="0">
-<segment>
-<pinref part="U1" gate="G$1" pin="P$1"/>
-<wire x1="73.66" y1="129.54" x2="63.5" y2="129.54" width="0.1524" layer="91"/>
-<label x="63.5" y="129.54" size="1.27" layer="95" rot="R180" xref="yes"/>
 </segment>
 </net>
@@
 </segment>
 </net>
-<net name="TRX_TX_SW" class="0">
-<segment>
-<pinref part="U1" gate="G$1" pin="P$4"/>
-<wire x1="73.66" y1="121.92" x2="63.5" y2="121.92" width="0.1524" layer="91"/>
-<label x="63.5" y="121.92" size="1.27" layer="95" rot="R180" xref="yes"/>
-</segment>
-</net>
