File: eagle/main.sch (EAGLE design)
At the start: 127 parts, among them IC1 LD117AS50TR, IC2 LD117AS33TR, IC3 OPA340U, Q1 BSS138, T3 AFT05MS004NT1, U1 STM32F777VIT, U3 L272, U4 ADAM TECH MCSP-Q1-08-A-SG, U5 SI4463-C2A-GM, U6 HMC546MS8GETR, X2 SMA, X3 ILSI 32MHz TCXO, X4 52746-0871

Commit message: Add files via upload
Connections:
- removed net +UB: C46.1, C47.1, C48.2, L7.2
- net +BATT: now also C46.1, C47.1, C48.2, L7.2
Changed lines of the file:
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@@
 <instance part="GND61" gate="1" x="127" y="124.46"/>
 <instance part="L7" gate="G$1" x="114.3" y="121.92" rot="R90"/>
-<instance part="SUPPLY3" gate="G$1" x="114.3" y="154.94"/>
+<instance part="SUPPLY3" gate="G$1" x="114.3" y="157.48"/>
 <instance part="+3V9" gate="G$1" x="226.06" y="162.56"/>
 <instance part="GND62" gate="1" x="226.06" y="127"/>
@@
 </segment>
 </net>
-<net name="+UB" class="0">
+<net name="N$28" class="0">
+<segment>
+<pinref part="R27" gate="G$1" pin="2"/>
+<pinref part="R29" gate="1" pin="A"/>
+</segment>
+</net>
+<net name="N$34" class="0">
+<segment>
+<pinref part="R28" gate="G$1" pin="1"/>
+<pinref part="R29" gate="1" pin="E"/>
+</segment>
+</net>
+<net name="+BATT" class="1">
 <segment>
 <pinref part="C46" gate="G$1" pin="1"/>
@@
 <junction x="114.3" y="144.78"/>
 <junction x="114.3" y="129.54"/>
-<wire x1="114.3" y1="149.86" x2="114.3" y2="152.4" width="0.1524" layer="91"/>
-<junction x="114.3" y="149.86"/>
 <pinref part="L7" gate="G$1" pin="2"/>
 <pinref part="SUPPLY3" gate="G$1" pin="+UB"/>
-</segment>
-</net>
-<net name="N$28" class="0">
-<segment>
-<pinref part="R27" gate="G$1" pin="2"/>
-<pinref part="R29" gate="1" pin="A"/>
-</segment>
-</net>
-<net name="N$34" class="0">
-<segment>
-<pinref part="R28" gate="G$1" pin="1"/>
-<pinref part="R29" gate="1" pin="E"/>
-</segment>
-</net>
+<wire x1="114.3" y1="149.86" x2="114.3" y2="154.94" width="0.1524" layer="91"/>
+<junction x="114.3" y="149.86"/>
+</segment>
+</net>
