File: eagle/kbd.sch (EAGLE design)
At the start: 29 parts, among them U1 STM32L011

Commit message: Add files via upload
Parts:
- added H1, H2, H3, H4, H5: MOUNT-PAD-ROUND2.8, holes:MOUNT-PAD-ROUND2.8
- JP1, JP2: device pinhead:PINHD-1X3/90 -> pinhead:PINHD-1X3
Connections:
- net GND: now also H1.MOUNT, H2.MOUNT, H3.MOUNT, H4.MOUNT, H5.MOUNT
