File: kicad/Mainboard/RF.sch (KiCad schematic (older format))
At the start: 95 parts, among them J7 Antenna, T1 AFT05MS004NT1, U5 HMC546MS8GETR

Commit message: Add files via upload
Parts:
- added R? (x2): 47k, symbol Device:R_Small
Connections:
- net +BATT: now also R?.2
- net GND: now also R?.1; no longer U?.5 (+), U?.6 (-)
- net at U?.7: now also U?.6 (-)
- new net: R?.1, R?.2, U?.5 (+)
Other:
- moved on the sheet: C?, U?C
Changed lines of the file:
@@
 $Descr A3 16535 11693
 encoding utf-8
-Sheet 5 7
+Sheet 5 8
 Title "RF circuit"
 Date ""
@@
 L Amplifier_Operational:LM2904 U?
 U 3 1 5E17FA82
-P 15700 4350
-F 0 "U?" H 15658 4396 50  0000 L CNN
-F 1 "LM2904" H 15658 4305 50  0000 L CNN
-F 2 "" H 15700 4350 50  0001 C CNN
-F 3 "http://www.ti.com/lit/ds/symlink/lm358.pdf" H 15700 4350 50  0001 C CNN
-	3    15700 4350
+P 14350 3300
+F 0 "U?" H 14308 3346 50  0000 L CNN
+F 1 "LM2904" H 14308 3255 50  0000 L CNN
+F 2 "" H 14350 3300 50  0001 C CNN
+F 3 "http://www.ti.com/lit/ds/symlink/lm358.pdf" H 14350 3300 50  0001 C CNN
+	3    14350 3300
 	1    0    0    -1
 $EndComp
@@
 L power:+BATT #PWR?
 U 1 1 5E187BBD
-P 15600 3850
-F 0 "#PWR?" H 15600 3700 50  0001 C CNN
-F 1 "+BATT" H 15615 4023 50  0000 C CNN
-F 2 "" H 15600 3850 50  0001 C CNN
-F 3 "" H 15600 3850 50  0001 C CNN
-	1    15600 3850
-	1    0    0    -1
-$EndComp
-Wire Wire Line
-	15600 3950 15600 4050
+P 14250 2800
+F 0 "#PWR?" H 14250 2650 50  0001 C CNN
+F 1 "+BATT" H 14265 2973 50  0000 C CNN
+F 2 "" H 14250 2800 50  0001 C CNN
+F 3 "" H 14250 2800 50  0001 C CNN
+	1    14250 2800
+	1    0    0    -1
+$EndComp
+Wire Wire Line
+	14250 2900 14250 3000
 $Comp
 L power:GND #PWR?
 U 1 1 5E18FAF9
-P 15600 4850
-F 0 "#PWR?" H 15600 4600 50  0001 C CNN
-F 1 "GND" H 15605 4677 50  0000 C CNN
-F 2 "" H 15600 4850 50  0001 C CNN
-F 3 "" H 15600 4850 50  0001 C CNN
-	1    15600 4850
-	1    0    0    -1
-$EndComp
-Wire Wire Line
-	15600 4650 15600 4750
+P 14250 3800
+F 0 "#PWR?" H 14250 3550 50  0001 C CNN
+F 1 "GND" H 14255 3627 50  0000 C CNN
+F 2 "" H 14250 3800 50  0001 C CNN
+F 3 "" H 14250 3800 50  0001 C CNN
+	1    14250 3800
+	1    0    0    -1
+$EndComp
+Wire Wire Line
+	14250 3600 14250 3700
 $Comp
 L Device:C_Small C?
@@
 L Device:C_Small C?
 U 1 1 5E1BF2C8
-P 15250 4400
-F 0 "C?" H 15342 4446 50  0000 L CNN
-F 1 "10n" H 15342 4355 50  0000 L CNN
-F 2 "" H 15250 4400 50  0001 C CNN
-F 3 "~" H 15250 4400 50  0001 C CNN
-	1    15250 4400
+P 13900 3350
+F 0 "C?" H 13992 3396 50  0000 L CNN
+F 1 "10n" H 13992 3305 50  0000 L CNN
+F 2 "" H 13900 3350 50  0001 C CNN
+F 3 "~" H 13900 3350 50  0001 C CNN
+	1    13900 3350
 	-1   0    0    -1
 $EndComp
 Wire Wire Line
-	15600 4750 15250 4750
-Wire Wire Line
-	15250 4750 15250 4500
-Wire Wire Line
-	15250 4300 15250 3950
-Wire Wire Line
-	15250 3950 15600 3950
-Wire Wire Line
-	15600 3950 15600 3850
-Connection ~ 15600 3950
-Wire Wire Line
-	15600 4750 15600 4850
-Connection ~ 15600 4750
+	14250 3700 13900 3700
+Wire Wire Line
+	13900 3700 13900 3450
+Wire Wire Line
+	13900 3250 13900 2900
+Wire Wire Line
+	13900 2900 14250 2900
+Wire Wire Line
+	14250 2900 14250 2800
+Connection ~ 14250 2900
+Wire Wire Line
+	14250 3700 14250 3800
+Connection ~ 14250 3700
 $Comp
 L power:GND #PWR?
 U 1 1 5E212E0D
-P 13500 6200
-F 0 "#PWR?" H 13500 5950 50  0001 C CNN
-F 1 "GND" H 13505 6027 50  0000 C CNN
-F 2 "" H 13500 6200 50  0001 C CNN
-F 3 "" H 13500 6200 50  0001 C CNN
-	1    13500 6200
-	1    0    0    -1
-$EndComp
-Wire Wire Line
-	13600 5800 13500 5800
-Wire Wire Line
-	13500 5800 13500 6000
-Wire Wire Line
-	13600 6000 13500 6000
-Connection ~ 13500 6000
-Wire Wire Line
-	13500 6000 13500 6200
+P 13300 6300
+F 0 "#PWR?" H 13300 6050 50  0001 C CNN
+F 1 "GND" H 13305 6127 50  0000 C CNN
+F 2 "" H 13300 6300 50  0001 C CNN
+F 3 "" H 13300 6300 50  0001 C CNN
+	1    13300 6300
+	1    0    0    -1
+$EndComp
 Wire Wire Line
 	14200 4300 14400 4300
@@
 Wire Wire Line
 	3050 6300 3150 6300
+$Comp
+L Device:R_Small R?
+U 1 1 5E27AFE6
+P 13300 5600
+F 0 "R?" V 13104 5600 50  0000 C CNN
+F 1 "47k" V 13195 5600 50  0000 C CNN
+F 2 "" H 13300 5600 50  0001 C CNN
+F 3 "~" H 13300 5600 50  0001 C CNN
+	1    13300 5600
+	-1   0    0    1
+$EndComp
+$Comp
+L Device:R_Small R?
+U 1 1 5E29428E
+P 13300 6200
+F 0 "R?" V 13104 6200 50  0000 C CNN
+F 1 "47k" V 13195 6200 50  0000 C CNN
+F 2 "" H 13300 6200 50  0001 C CNN
+F 3 "~" H 13300 6200 50  0001 C CNN
+	1    13300 6200
+	-1   0    0    1
+$EndComp
+$Comp
+L power:+BATT #PWR?
+U 1 1 5E2E4147
+P 13300 5500
+F 0 "#PWR?" H 13300 5350 50  0001 C CNN
+F 1 "+BATT" H 13315 5673 50  0000 C CNN
+F 2 "" H 13300 5500 50  0001 C CNN
+F 3 "" H 13300 5500 50  0001 C CNN
+	1    13300 5500
+	1    0    0    -1
+$EndComp
+Wire Wire Line
+	13300 5700 13300 5800
+Wire Wire Line
+	13600 6000 13550 6000
+Wire Wire Line
+	13550 6000 13550 6200
+Wire Wire Line
+	13550 6200 14300 6200
+Wire Wire Line
+	14300 6200 14300 5900
+Wire Wire Line
+	14300 5900 14200 5900
+Wire Wire Line
+	13300 5800 13300 6100
+Connection ~ 13300 5800
+Wire Wire Line
+	13300 5800 13600 5800
 $EndSCHEMATC

Commit message: Add files via upload
Connections:
- net ADF_CLKOUT renamed SPI1_SCK
- net ADF_DATAIN renamed SPI2_MISO
- net ADF_DATAOUT renamed SPI2_MOSI
Changed lines of the file:
@@
 Wire Wire Line
 	6600 8450 6700 8450
-Text GLabel 6700 8250 2    50   Input ~ 0
-ADF_CLKOUT
-Text GLabel 6700 8350 2    50   Input ~ 0
-ADF_DATAIN
-Text GLabel 6700 8450 2    50   Input ~ 0
-ADF_DATAOUT
 $Comp
 L Device:C_Small C?
@@
 Wire Wire Line
 	6250 9350 6350 9350
-Text GLabel 6350 9050 2    50   Input ~ 0
+Text GLabel 6350 9050 2    50   Input ~ 10
 ADF_SCLK
-Text GLabel 6350 9150 2    50   Input ~ 0
+Text GLabel 6350 9150 2    50   Input ~ 10
 ADF_SREAD
-Text GLabel 6350 9250 2    50   Input ~ 0
+Text GLabel 6350 9250 2    50   Input ~ 10
 ADF_SDATA
-Text GLabel 6350 9350 2    50   Input ~ 0
+Text GLabel 6350 9350 2    50   Input ~ 10
 ADF_SLE
 Wire Wire Line
@@
 Wire Wire Line
 	5750 10000 5850 10000
-Text GLabel 5850 10000 2    50   Input ~ 0
+Text GLabel 5850 10000 2    50   Input ~ 10
 ADF_CE
 NoConn ~ 5650 9900
@@
 Wire Wire Line
 	6250 8550 6700 8550
-Text GLabel 6700 8550 2    50   Output ~ 0
+Text GLabel 6700 8550 2    50   Output ~ 10
 ADF_SWD
 $Comp
@@
 Wire Wire Line
 	3650 6300 3550 6300
-Text GLabel 2550 6300 0    50   Input ~ 0
+Text GLabel 2550 6300 0    50   Input ~ 10
 FM_MOD
 Text Notes 4350 5700 2    50   ~ 0
@@
 Wire Wire Line
 	13300 5800 13600 5800
+Text GLabel 6700 8250 2    50   Input ~ 10
+SPI1_SCK
+Text GLabel 6700 8350 2    50   Input ~ 10
+SPI2_MISO
+Text GLabel 6700 8450 2    50   Input ~ 10
+SPI2_MOSI
 $EndSCHEMATC
