File: kicad/Mainboard/STM32.sch (KiCad schematic (older format))
At the start: 21 parts, among them J1 SWD, J2 USB_OTG, J3 TP1, J4 TP2, U1 STM32F777VIT, U2 USBLC6-2SC6

Commit message: Updated WIP schematics
Parts:
- added Q?: BC847, Package_TO_SOT_SMD:SOT-23, symbol Transistor_BJT:BC847
- added R?: 1k, symbol Device:R_Small
- added R?: 10k, symbol Device:R_Small
Connections:
- net labels added: PTT
- net labels removed: PTT_EXT, PTT_IN
- wire segments 131 -> 136
- no-connect marks 42 -> 43
Other:
- moved on the sheet: R4
Changed lines of the file:
@@
 BOOT0
 Text GLabel 4100 1450 1    50   Input ~ 10
-PTT_IN
+PTT
 $Comp
 L power:GND #PWR05
@@
 L Mainboard-rescue:R_Small-device R4
 U 1 1 5DEC41C2
-P 1450 5800
-F 0 "R4" H 1509 5846 50  0000 L CNN
-F 1 "10k" H 1509 5755 50  0000 L CNN
-F 2 "" H 1450 5800 50  0001 C CNN
-F 3 "~" H 1450 5800 50  0001 C CNN
-	1    1450 5800
-	1    0    0    -1
-$EndComp
-Text GLabel 1200 5600 1    50   Input ~ 10
+P 2450 6400
+F 0 "R4" H 2509 6446 50  0000 L CNN
+F 1 "10k" H 2509 6355 50  0000 L CNN
+F 2 "" H 2450 6400 50  0001 C CNN
+F 3 "~" H 2450 6400 50  0001 C CNN
+	1    2450 6400
+	1    0    0    -1
+$EndComp
+Text GLabel 1900 6600 2    50   Input ~ 10
 BOOT0
 $Comp
 L power:+3V3 #PWR020
 U 1 1 5DEC8A28
-P 1450 5600
-F 0 "#PWR020" H 1450 5450 50  0001 C CNN
-F 1 "+3V3" H 1465 5773 50  0000 C CNN
-F 2 "" H 1450 5600 50  0001 C CNN
-F 3 "" H 1450 5600 50  0001 C CNN
-	1    1450 5600
-	1    0    0    -1
-$EndComp
-Wire Wire Line
-	1450 5600 1450 5700
-Wire Wire Line
-	1450 5900 1450 6000
-Text GLabel 1450 6000 3    50   Input ~ 10
+P 2450 6200
+F 0 "#PWR020" H 2450 6050 50  0001 C CNN
+F 1 "+3V3" H 2465 6373 50  0000 C CNN
+F 2 "" H 2450 6200 50  0001 C CNN
+F 3 "" H 2450 6200 50  0001 C CNN
+	1    2450 6200
+	1    0    0    -1
+$EndComp
+Wire Wire Line
+	2450 6200 2450 6300
+Wire Wire Line
+	2450 6500 2450 6600
+Text GLabel 2450 6600 3    50   Input ~ 10
 NRST
 $Comp
@@
 Wire Wire Line
 	6900 2750 7100 2750
-Text GLabel 1200 6000 3    50   Input ~ 10
-PTT_IN
-Wire Wire Line
-	1200 5600 1200 6000
+Text GLabel 1100 6900 0    50   Input ~ 10
+PTT
 Wire Wire Line
 	8450 5400 8650 5400
@@
 	1    0    0    -1
 $EndComp
-Wire Wire Line
-	4000 1550 4000 1450
-Text GLabel 4000 1450 1    50   Input ~ 10
-PTT_EXT
 NoConn ~ 4200 1550
+$Comp
+L Device:R_Small R?
+U 1 1 5E0DF68A
+P 1300 6900
+F 0 "R?" V 1104 6900 50  0000 C CNN
+F 1 "1k" V 1195 6900 50  0000 C CNN
+F 2 "" H 1300 6900 50  0001 C CNN
+F 3 "~" H 1300 6900 50  0001 C CNN
+	1    1300 6900
+	0    1    1    0
+$EndComp
+Wire Wire Line
+	1400 6900 1500 6900
+Wire Wire Line
+	1100 6900 1200 6900
+$Comp
+L Transistor_BJT:BC847 Q?
+U 1 1 5E0E8B40
+P 1700 6900
+F 0 "Q?" H 1891 6946 50  0000 L CNN
+F 1 "BC847" H 1891 6855 50  0000 L CNN
+F 2 "Package_TO_SOT_SMD:SOT-23" H 1900 6825 50  0001 L CIN
+F 3 "http://www.infineon.com/dgdl/Infineon-BC847SERIES_BC848SERIES_BC849SERIES_BC850SERIES-DS-v01_01-en.pdf?fileId=db3a304314dca389011541d4630a1657" H 1700 6900 50  0001 L CNN
+	1    1700 6900
+	1    0    0    -1
+$EndComp
+Wire Wire Line
+	1900 6600 1800 6600
+Wire Wire Line
+	1800 6600 1800 6700
+$Comp
+L Device:R_Small R?
+U 1 1 5E0EDCC6
+P 1800 6400
+F 0 "R?" H 1741 6354 50  0000 R CNN
+F 1 "10k" H 1741 6445 50  0000 R CNN
+F 2 "" H 1800 6400 50  0001 C CNN
+F 3 "~" H 1800 6400 50  0001 C CNN
+	1    1800 6400
+	1    0    0    1
+$EndComp
+Wire Wire Line
+	1800 6500 1800 6600
+Connection ~ 1800 6600
+$Comp
+L power:+3V3 #PWR?
+U 1 1 5E0F302C
+P 1800 6200
+F 0 "#PWR?" H 1800 6050 50  0001 C CNN
+F 1 "+3V3" H 1815 6373 50  0000 C CNN
+F 2 "" H 1800 6200 50  0001 C CNN
+F 3 "" H 1800 6200 50  0001 C CNN
+	1    1800 6200
+	1    0    0    -1
+$EndComp
+Wire Wire Line
+	1800 6200 1800 6300
+$Comp
+L power:GND #PWR?
+U 1 1 5E0F8338
+P 1800 7200
+F 0 "#PWR?" H 1800 6950 50  0001 C CNN
+F 1 "GND" H 1805 7027 50  0000 C CNN
+F 2 "" H 1800 7200 50  0001 C CNN
+F 3 "" H 1800 7200 50  0001 C CNN
+	1    1800 7200
+	1    0    0    -1
+$EndComp
+Wire Wire Line
+	1800 7100 1800 7200
+NoConn ~ 4000 1550
 $EndSCHEMATC

Commit message: Add files via upload
* replaced Q7 with BSS138
* new HMI connector (for keypad and display)
Parts:
- removed Q?: BC847, Package_TO_SOT_SMD:SOT-23, symbol Transistor_BJT:BC847
- removed R?: 1k, symbol Device:R_Small
- added Q?: BSS138, Package_TO_SOT_SMD:SOT-23, symbol Transistor_FET:BSS138
Connections:
- net labels removed: TFT_A0
- wire segments 136 -> 134
Other:
- note added: "TODO: \n* add PWR_ON signal for the GPS module\n* add pin names/functions"
- note removed: "TODO: \n* add PWR_ON signal for the GPS module\n* Add pin names/functions"
Changed lines of the file:
@@
 EESchema Schematic File Version 4
+LIBS:Mainboard-cache
 EELAYER 30 0
 EELAYER END
@@
 Text GLabel 7100 3350 2    50   Input ~ 10
 TFT_RST
-Text GLabel 7100 3450 2    50   Input ~ 10
-TFT_A0
 Text GLabel 7100 3850 2    50   Input ~ 10
 BLIGHT_CTRL
@@
 Wire Wire Line
 	6900 3350 7100 3350
-Wire Wire Line
-	6900 3450 7100 3450
 Wire Wire Line
 	6900 3850 7100 3850
@@
 	8300 1150 8400 1150
 Text Notes 3600 2850 0    50   ~ 10
-TODO: \n* add PWR_ON signal for the GPS module\n* Add pin names/functions
+TODO: \n* add PWR_ON signal for the GPS module\n* add pin names/functions
 $Comp
 L Mainboard-rescue:USBLC6-2SC6-ESD_Protection U2
@@
 Wire Wire Line
 	6900 2750 7100 2750
-Text GLabel 1100 6900 0    50   Input ~ 10
+Text GLabel 1300 6900 0    50   Input ~ 10
 PTT
 Wire Wire Line
@@
 $EndComp
 NoConn ~ 4200 1550
-$Comp
-L Device:R_Small R?
-U 1 1 5E0DF68A
-P 1300 6900
-F 0 "R?" V 1104 6900 50  0000 C CNN
-F 1 "1k" V 1195 6900 50  0000 C CNN
-F 2 "" H 1300 6900 50  0001 C CNN
-F 3 "~" H 1300 6900 50  0001 C CNN
-	1    1300 6900
-	0    1    1    0
-$EndComp
-Wire Wire Line
-	1400 6900 1500 6900
-Wire Wire Line
-	1100 6900 1200 6900
-$Comp
-L Transistor_BJT:BC847 Q?
-U 1 1 5E0E8B40
-P 1700 6900
-F 0 "Q?" H 1891 6946 50  0000 L CNN
-F 1 "BC847" H 1891 6855 50  0000 L CNN
-F 2 "Package_TO_SOT_SMD:SOT-23" H 1900 6825 50  0001 L CIN
-F 3 "http://www.infineon.com/dgdl/Infineon-BC847SERIES_BC848SERIES_BC849SERIES_BC850SERIES-DS-v01_01-en.pdf?fileId=db3a304314dca389011541d4630a1657" H 1700 6900 50  0001 L CNN
-	1    1700 6900
-	1    0    0    -1
-$EndComp
 Wire Wire Line
 	1900 6600 1800 6600
@@
 	1800 7100 1800 7200
 NoConn ~ 4000 1550
+$Comp
+L Transistor_FET:BSS138 Q?
+U 1 1 5E22ECEC
+P 1700 6900
+F 0 "Q?" H 1906 6946 50  0000 L CNN
+F 1 "BSS138" H 1906 6855 50  0000 L CNN
+F 2 "Package_TO_SOT_SMD:SOT-23" H 1900 6825 50  0001 L CIN
+F 3 "https://www.fairchildsemi.com/datasheets/BS/BSS138.pdf" H 1700 6900 50  0001 L CNN
+	1    1700 6900
+	1    0    0    -1
+$EndComp
+Wire Wire Line
+	1500 6900 1300 6900
 $EndSCHEMATC

Commit message: Add files via upload
Connections:
- net BLIGHT_CTRL: now also U1.91 (P$91); no longer U1.59 (P$59)
- net SPI1_CS: now also U1.90 (P$90); no longer U1.32 (P$32)
- net SPI1_MOSI: now also U1.88 (P$88); no longer U1.31 (P$31)
- net SPI1_SCK: now also U1.89 (P$89); no longer U1.29 (P$29)
- net TFT_RST: now also U1.85 (P$85); no longer U1.64 (P$64)
- net ADC3_1: now reaches U1.23 (P$23)
- net GPS_EN: now reaches U1.67 (P$67)
- net DAC_OUT renamed AUDIO_DAC
- net SPI1_MISO: no longer names the net of U1.30 (P$30)
- net TRX_NIRQ: no longer names the net of U1.35 (P$35)
- net TRX_SDN: no longer names the net of U1.34 (P$34)
- new net PA_RAMP: U1.29 (P$29)
- no-connect marks 43 -> 44
Other:
- note added: "ADC1_0 Microphone input\nADC3_1 FM demod input\nADC2_3 Battery voltage monitor"
- moved on the sheet: J1
Changed lines of the file:
@@
 EESchema Schematic File Version 4
+LIBS:Mainboard-cache
 EELAYER 30 0
 EELAYER END
@@
 NoConn ~ 3100 3850
 NoConn ~ 3100 3950
-NoConn ~ 3100 4450
 NoConn ~ 3100 4550
 $Comp
@@
 	6350 5500 6350 5400
 Text GLabel 4000 5450 3    50   Input ~ 10
-DAC_OUT
-Text GLabel 4100 5450 3    50   Input ~ 10
-SPI1_SCK
-Text GLabel 4200 5450 3    50   Input ~ 10
-SPI1_MISO
-Text GLabel 4300 5450 3    50   Input ~ 10
-SPI1_MOSI
-Text GLabel 4400 5450 3    50   Input ~ 10
-SPI1_CS
-Text GLabel 4600 5450 3    50   Input ~ 10
-TRX_SDN
-Text GLabel 4700 5450 3    50   Input ~ 10
-TRX_NIRQ
+AUDIO_DAC
 Text GLabel 5800 5450 3    50   Input ~ 10
 USART3_TX
@@
 Wire Wire Line
 	4000 5350 4000 5450
-Wire Wire Line
-	4100 5350 4100 5450
-Wire Wire Line
-	4200 5350 4200 5450
-Wire Wire Line
-	4300 5350 4300 5450
-Wire Wire Line
-	4400 5350 4400 5450
-Wire Wire Line
-	4600 5350 4600 5450
-Wire Wire Line
-	4700 5350 4700 5450
 Wire Wire Line
 	5800 5350 5800 5450
@@
 Text GLabel 7100 3250 2    50   Input ~ 10
 SD_D0
-Text GLabel 7100 3350 2    50   Input ~ 10
+Text GLabel 5300 1450 1    50   Input ~ 10
 TFT_RST
-Text GLabel 7100 3850 2    50   Input ~ 10
+Text GLabel 4700 1450 1    50   Input ~ 10
 BLIGHT_CTRL
 Text GLabel 7100 4250 2    50   Input ~ 10
@@
 	6900 3250 7100 3250
 Wire Wire Line
-	6900 3350 7100 3350
-Wire Wire Line
-	6900 3850 7100 3850
-Wire Wire Line
 	6900 4250 7100 4250
 Wire Wire Line
@@
 Wire Wire Line
 	7750 2750 7750 2850
-NoConn ~ 6900 3050
 NoConn ~ 6900 3550
 NoConn ~ 6900 3650
@@
 	6200 1450 6200 1550
 NoConn ~ 4300 1550
-NoConn ~ 4700 1550
-NoConn ~ 4800 1550
-NoConn ~ 4900 1550
-NoConn ~ 5000 1550
-NoConn ~ 5300 1550
 NoConn ~ 5400 1550
 NoConn ~ 6100 1550
@@
 L Mainboard-rescue:Conn_01x05-conn J1
 U 1 1 5DECD704
-P 8100 1050
-F 0 "J1" H 8018 625 50  0000 C CNN
-F 1 "SWD" H 8018 716 50  0000 C CNN
-F 2 "" H 8100 1050 50  0001 C CNN
-F 3 "~" H 8100 1050 50  0001 C CNN
-	1    8100 1050
+P 7900 1300
+F 0 "J1" H 7818 875 50  0000 C CNN
+F 1 "SWD" H 7818 966 50  0000 C CNN
+F 2 "" H 7900 1300 50  0001 C CNN
+F 3 "~" H 7900 1300 50  0001 C CNN
+	1    7900 1300
 	-1   0    0    1
 $EndComp
@@
 L power:+3V3 #PWR02
 U 1 1 5DECE401
-P 8400 750
-F 0 "#PWR02" H 8400 600 50  0001 C CNN
-F 1 "+3V3" H 8415 923 50  0000 C CNN
-F 2 "" H 8400 750 50  0001 C CNN
-F 3 "" H 8400 750 50  0001 C CNN
-	1    8400 750
-	1    0    0    -1
-$EndComp
-Wire Wire Line
-	8300 850  8400 850
-Wire Wire Line
-	8400 850  8400 750
+P 8200 1000
+F 0 "#PWR02" H 8200 850 50  0001 C CNN
+F 1 "+3V3" H 8215 1173 50  0000 C CNN
+F 2 "" H 8200 1000 50  0001 C CNN
+F 3 "" H 8200 1000 50  0001 C CNN
+	1    8200 1000
+	1    0    0    -1
+$EndComp
+Wire Wire Line
+	8100 1100 8200 1100
+Wire Wire Line
+	8200 1100 8200 1000
 $Comp
 L power:GND #PWR04
 U 1 1 5DED1019
-P 8400 1350
-F 0 "#PWR04" H 8400 1100 50  0001 C CNN
-F 1 "GND" H 8405 1177 50  0000 C CNN
-F 2 "" H 8400 1350 50  0001 C CNN
-F 3 "" H 8400 1350 50  0001 C CNN
-	1    8400 1350
-	1    0    0    -1
-$EndComp
-Wire Wire Line
-	8300 1250 8400 1250
-Wire Wire Line
-	8400 1250 8400 1350
-Text GLabel 8400 950  2    50   Input ~ 10
+P 8200 1600
+F 0 "#PWR04" H 8200 1350 50  0001 C CNN
+F 1 "GND" H 8205 1427 50  0000 C CNN
+F 2 "" H 8200 1600 50  0001 C CNN
+F 3 "" H 8200 1600 50  0001 C CNN
+	1    8200 1600
+	1    0    0    -1
+$EndComp
+Wire Wire Line
+	8100 1500 8200 1500
+Wire Wire Line
+	8200 1500 8200 1600
+Text GLabel 8200 1200 2    50   Input ~ 10
 SWDIO
-Text GLabel 8400 1050 2    50   Input ~ 10
+Text GLabel 8200 1300 2    50   Input ~ 10
 SWCLK
-Text GLabel 8400 1150 2    50   Input ~ 10
+Text GLabel 8200 1400 2    50   Input ~ 10
 NRST
 Wire Wire Line
-	8300 950  8400 950
-Wire Wire Line
-	8300 1050 8400 1050
-Wire Wire Line
-	8300 1150 8400 1150
+	8100 1200 8200 1200
+Wire Wire Line
+	8100 1300 8200 1300
+Wire Wire Line
+	8100 1400 8200 1400
 Text Notes 3600 2850 0    50   ~ 10
 TODO: \n* add PWR_ON signal for the GPS module\n* add pin names/functions
@@
 Wire Wire Line
 	1500 6900 1300 6900
+Wire Wire Line
+	4100 5450 4100 5350
+Text GLabel 4100 5450 3    50   Input ~ 10
+PA_RAMP
+Wire Wire Line
+	2800 4450 3100 4450
+Text GLabel 2800 4450 0    50   Input ~ 10
+ADC3_1
+Text Notes 850  4600 0    50   ~ 0
+ADC1_0    Microphone input\nADC3_1    FM demod input\nADC2_3    Battery voltage monitor
+Wire Notes Line
+	850  4350 2250 4350
+Wire Notes Line
+	2250 4350 2250 4600
+Wire Notes Line
+	2250 4600 850  4600
+Wire Notes Line
+	850  4600 850  4350
+NoConn ~ 4600 5350
+NoConn ~ 4700 5350
+NoConn ~ 4200 5350
+NoConn ~ 4300 5350
+NoConn ~ 4400 5350
+Wire Wire Line
+	4800 1450 4800 1550
+Wire Wire Line
+	4900 1450 4900 1550
+Wire Wire Line
+	5000 1450 5000 1550
+Text GLabel 4800 1450 1    50   Input ~ 10
+SPI1_CS
+Text GLabel 4900 1450 1    50   Input ~ 10
+SPI1_SCK
+Text GLabel 5000 1450 1    50   Input ~ 10
+SPI1_MOSI
+Wire Wire Line
+	7100 3050 6900 3050
+Text GLabel 7100 3050 2    50   Input ~ 10
+GPS_EN
+Wire Wire Line
+	4700 1450 4700 1550
+Wire Wire Line
+	5300 1450 5300 1550
+NoConn ~ 6900 3350
+NoConn ~ 6900 3450
+NoConn ~ 6900 3850
 $EndSCHEMATC

Commit message: Add files via upload
Connections:
- net SPK_AMP_SEL: now reaches U1.34 (P$34)
- net FM_MOD_SEL: now reaches U1.35 (P$35)
- no-connect marks 44 -> 42
Changed lines of the file:
@@
 Text GLabel 2800 4450 0    50   Input ~ 10
 ADC3_1
-Text Notes 850  4600 0    50   ~ 0
-ADC1_0    Microphone input\nADC3_1    FM demod input\nADC2_3    Battery voltage monitor
+Text Notes 800  4550 0    50   ~ 0
+ADC1_0  Microphone input\nADC3_1  FM demod input\nADC2_3  Battery voltage monitor
 Wire Notes Line
-	850  4350 2250 4350
+	800  4300 2200 4300
 Wire Notes Line
-	2250 4350 2250 4600
+	2200 4300 2200 4550
 Wire Notes Line
-	2250 4600 850  4600
+	2200 4550 800  4550
 Wire Notes Line
-	850  4600 850  4350
-NoConn ~ 4600 5350
-NoConn ~ 4700 5350
+	800  4550 800  4300
 NoConn ~ 4200 5350
 NoConn ~ 4300 5350
@@
 NoConn ~ 6900 3450
 NoConn ~ 6900 3850
+Wire Wire Line
+	4600 5450 4600 5350
+Wire Wire Line
+	4700 5450 4700 5350
+Text GLabel 4600 5450 3    50   Input ~ 10
+SPK_AMP_SEL
+Text GLabel 4700 5450 3    50   Input ~ 10
+FM_MOD_SEL
 $EndSCHEMATC

Commit message: Add files via upload
Connections:
- net UART7_RX: now reaches U1.37 (P$37)
- net UART7_TX: now reaches U1.38 (P$38)
- net WIFI_EN: now reaches U1.45 (P$45)
- no-connect marks 42 -> 39
Other:
- note added: "TODO:\n* add pin names/functions"
- note added: "USART1 GPS\nUSART2 Debug\nUSART3 ESP8266-12\nUSART7 HMI"
- note removed: "TODO: \n* add PWR_ON signal for the GPS module\n* add pin names/functions"
- moved on the sheet: C1, C2, FB1, FB2, J1, J3, J4
Changed lines of the file:
@@
 $Descr A4 11693 8268
 encoding utf-8
-Sheet 2 7
+Sheet 2 8
 Title "Microcontroller"
 Date ""
@@
 L Mainboard-rescue:Ferrite_Bead_Small-device FB1
 U 1 1 5DE315C2
-P 800 850
-F 0 "FB1" V 563 850 50  0000 C CNN
-F 1 "TBD" V 654 850 50  0000 C CNN
-F 2 "" V 730 850 50  0001 C CNN
-F 3 "~" H 800 850 50  0001 C CNN
-	1    800  850
+P 1200 1150
+F 0 "FB1" V 963 1150 50  0000 C CNN
+F 1 "TBD" V 1054 1150 50  0000 C CNN
+F 2 "" V 1130 1150 50  0001 C CNN
+F 3 "~" H 1200 1150 50  0001 C CNN
+	1    1200 1150
 	0    1    1    0
 $EndComp
@@
 L Mainboard-rescue:Ferrite_Bead_Small-device FB2
 U 1 1 5DE31FCE
-P 800 1250
-F 0 "FB2" V 563 1250 50  0000 C CNN
-F 1 "TBD" V 654 1250 50  0000 C CNN
-F 2 "" V 730 1250 50  0001 C CNN
-F 3 "~" H 800 1250 50  0001 C CNN
-	1    800  1250
+P 1200 1550
+F 0 "FB2" V 963 1550 50  0000 C CNN
+F 1 "TBD" V 1054 1550 50  0000 C CNN
+F 2 "" V 1130 1550 50  0001 C CNN
+F 3 "~" H 1200 1550 50  0001 C CNN
+	1    1200 1550
 	0    1    1    0
 $EndComp
@@
 L Mainboard-rescue:C_Small-device C1
 U 1 1 5DE325EB
-P 1000 1450
-F 0 "C1" H 1092 1496 50  0000 L CNN
-F 1 "100n" H 1092 1405 50  0000 L CNN
-F 2 "" H 1000 1450 50  0001 C CNN
-F 3 "~" H 1000 1450 50  0001 C CNN
-	1    1000 1450
+P 1400 1750
+F 0 "C1" H 1492 1796 50  0000 L CNN
+F 1 "100n" H 1492 1705 50  0000 L CNN
+F 2 "" H 1400 1750 50  0001 C CNN
+F 3 "~" H 1400 1750 50  0001 C CNN
+	1    1400 1750
 	1    0    0    -1
 $EndComp
@@
 L Mainboard-rescue:C_Small-device C2
 U 1 1 5DE32C17
-P 1400 1450
-F 0 "C2" H 1492 1496 50  0000 L CNN
-F 1 "100n" H 1492 1405 50  0000 L CNN
-F 2 "" H 1400 1450 50  0001 C CNN
-F 3 "~" H 1400 1450 50  0001 C CNN
-	1    1400 1450
-	1    0    0    -1
-$EndComp
-Wire Wire Line
-	900  1250 1000 1250
-Wire Wire Line
-	1000 1250 1000 1350
-Wire Wire Line
-	900  850  1400 850
-Wire Wire Line
-	1400 850  1400 1350
-Wire Wire Line
-	600  750  600  850
-Wire Wire Line
-	600  850  700  850
-Wire Wire Line
-	600  850  600  1250
-Wire Wire Line
-	600  1250 700  1250
-Connection ~ 600  850
+P 1800 1750
+F 0 "C2" H 1892 1796 50  0000 L CNN
+F 1 "100n" H 1892 1705 50  0000 L CNN
+F 2 "" H 1800 1750 50  0001 C CNN
+F 3 "~" H 1800 1750 50  0001 C CNN
+	1    1800 1750
+	1    0    0    -1
+$EndComp
+Wire Wire Line
+	1300 1550 1400 1550
+Wire Wire Line
+	1400 1550 1400 1650
+Wire Wire Line
+	1300 1150 1800 1150
+Wire Wire Line
+	1800 1150 1800 1650
+Wire Wire Line
+	1000 1050 1000 1150
+Wire Wire Line
+	1000 1150 1100 1150
+Wire Wire Line
+	1000 1150 1000 1550
+Wire Wire Line
+	1000 1550 1100 1550
+Connection ~ 1000 1150
 $Comp
 L power:GND #PWR06
 U 1 1 5DE33EB8
-P 1000 1650
-F 0 "#PWR06" H 1000 1400 50  0001 C CNN
-F 1 "GND" H 1005 1477 50  0000 C CNN
-F 2 "" H 1000 1650 50  0001 C CNN
-F 3 "" H 1000 1650 50  0001 C CNN
-	1    1000 1650
+P 1400 1950
+F 0 "#PWR06" H 1400 1700 50  0001 C CNN
+F 1 "GND" H 1405 1777 50  0000 C CNN
+F 2 "" H 1400 1950 50  0001 C CNN
+F 3 "" H 1400 1950 50  0001 C CNN
+	1    1400 1950
 	1    0    0    -1
 $EndComp
@@
 L power:+3V3 #PWR01
 U 1 1 5DE34250
-P 600 750
-F 0 "#PWR01" H 600 600 50  0001 C CNN
-F 1 "+3V3" H 615 923 50  0000 C CNN
-F 2 "" H 600 750 50  0001 C CNN
-F 3 "" H 600 750 50  0001 C CNN
-	1    600  750
+P 1000 1050
+F 0 "#PWR01" H 1000 900 50  0001 C CNN
+F 1 "+3V3" H 1015 1223 50  0000 C CNN
+F 2 "" H 1000 1050 50  0001 C CNN
+F 3 "" H 1000 1050 50  0001 C CNN
+	1    1000 1050
 	1    0    0    -1
 $EndComp
@@
 L power:GND #PWR07
 U 1 1 5DE35163
-P 1400 1650
-F 0 "#PWR07" H 1400 1400 50  0001 C CNN
-F 1 "GND" H 1405 1477 50  0000 C CNN
-F 2 "" H 1400 1650 50  0001 C CNN
-F 3 "" H 1400 1650 50  0001 C CNN
-	1    1400 1650
-	1    0    0    -1
-$EndComp
-Wire Wire Line
-	1400 1550 1400 1650
-Wire Wire Line
-	1000 1550 1000 1650
-Wire Wire Line
-	1400 850  1500 850
-Connection ~ 1400 850
-Wire Wire Line
-	1000 1250 1500 1250
-Connection ~ 1000 1250
-Text GLabel 1500 850  2    50   Input ~ 10
+P 1800 1950
+F 0 "#PWR07" H 1800 1700 50  0001 C CNN
+F 1 "GND" H 1805 1777 50  0000 C CNN
+F 2 "" H 1800 1950 50  0001 C CNN
+F 3 "" H 1800 1950 50  0001 C CNN
+	1    1800 1950
+	1    0    0    -1
+$EndComp
+Wire Wire Line
+	1800 1850 1800 1950
+Wire Wire Line
+	1400 1850 1400 1950
+Wire Wire Line
+	1800 1150 1900 1150
+Connection ~ 1800 1150
+Wire Wire Line
+	1400 1550 1900 1550
+Connection ~ 1400 1550
+Text GLabel 1900 1150 2    50   Input ~ 10
 VREF
-Text GLabel 1500 1250 2    50   Input ~ 10
+Text GLabel 1900 1550 2    50   Input ~ 10
 VDDA
 $Comp
@@
 L Mainboard-rescue:TEST_1P-conn J3
 U 1 1 5DE542F9
-P 5100 5450
-F 0 "J3" V 5200 5600 50  0000 R CNN
-F 1 "TP1" V 5200 5750 50  0000 R CNN
-F 2 "" H 5300 5450 50  0001 C CNN
-F 3 "" H 5300 5450 50  0001 C CNN
-	1    5100 5450
+P 5100 5950
+F 0 "J3" V 5200 6100 50  0000 R CNN
+F 1 "TP1" V 5200 6250 50  0000 R CNN
+F 2 "" H 5300 5950 50  0001 C CNN
+F 3 "" H 5300 5950 50  0001 C CNN
+	1    5100 5950
 	-1   0    0    1
 $EndComp
@@
 L Mainboard-rescue:TEST_1P-conn J4
 U 1 1 5DE55232
-P 5200 5450
-F 0 "J4" V 5300 5600 50  0000 R CNN
-F 1 "TP2" V 5300 5750 50  0000 R CNN
-F 2 "" H 5400 5450 50  0001 C CNN
-F 3 "" H 5400 5450 50  0001 C CNN
-	1    5200 5450
+P 5200 5950
+F 0 "J4" V 5300 6100 50  0000 R CNN
+F 1 "TP2" V 5300 6250 50  0000 R CNN
+F 2 "" H 5400 5950 50  0001 C CNN
+F 3 "" H 5400 5950 50  0001 C CNN
+	1    5200 5950
 	1    0    0    1
 $EndComp
-Wire Wire Line
-	5100 5350 5100 5450
-Wire Wire Line
-	5200 5350 5200 5450
 $Comp
 L Mainboard-rescue:C_Small-device C7
@@
 NoConn ~ 4500 5350
 NoConn ~ 4800 5350
-NoConn ~ 4900 5350
-NoConn ~ 5000 5350
 NoConn ~ 5300 5350
 NoConn ~ 5400 5350
 NoConn ~ 5500 5350
 NoConn ~ 5600 5350
-NoConn ~ 5700 5350
 Wire Wire Line
 	6900 2350 7000 2350
@@
 L Mainboard-rescue:Conn_01x05-conn J1
 U 1 1 5DECD704
-P 7900 1300
-F 0 "J1" H 7818 875 50  0000 C CNN
-F 1 "SWD" H 7818 966 50  0000 C CNN
-F 2 "" H 7900 1300 50  0001 C CNN
-F 3 "~" H 7900 1300 50  0001 C CNN
-	1    7900 1300
+P 9250 3350
+F 0 "J1" H 9168 2925 50  0000 C CNN
+F 1 "SWD" H 9168 3016 50  0000 C CNN
+F 2 "" H 9250 3350 50  0001 C CNN
+F 3 "~" H 9250 3350 50  0001 C CNN
+	1    9250 3350
 	-1   0    0    1
 $EndComp
@@
 L power:+3V3 #PWR02
 U 1 1 5DECE401
-P 8200 1000
-F 0 "#PWR02" H 8200 850 50  0001 C CNN
-F 1 "+3V3" H 8215 1173 50  0000 C CNN
-F 2 "" H 8200 1000 50  0001 C CNN
-F 3 "" H 8200 1000 50  0001 C CNN
-	1    8200 1000
-	1    0    0    -1
-$EndComp
-Wire Wire Line
-	8100 1100 8200 1100
-Wire Wire Line
-	8200 1100 8200 1000
+P 9550 3050
+F 0 "#PWR02" H 9550 2900 50  0001 C CNN
+F 1 "+3V3" H 9565 3223 50  0000 C CNN
+F 2 "" H 9550 3050 50  0001 C CNN
+F 3 "" H 9550 3050 50  0001 C CNN
+	1    9550 3050
+	1    0    0    -1
+$EndComp
+Wire Wire Line
+	9450 3150 9550 3150
+Wire Wire Line
+	9550 3150 9550 3050
 $Comp
 L power:GND #PWR04
 U 1 1 5DED1019
-P 8200 1600
-F 0 "#PWR04" H 8200 1350 50  0001 C CNN
-F 1 "GND" H 8205 1427 50  0000 C CNN
-F 2 "" H 8200 1600 50  0001 C CNN
-F 3 "" H 8200 1600 50  0001 C CNN
-	1    8200 1600
-	1    0    0    -1
-$EndComp
-Wire Wire Line
-	8100 1500 8200 1500
-Wire Wire Line
-	8200 1500 8200 1600
-Text GLabel 8200 1200 2    50   Input ~ 10
+P 9550 3650
+F 0 "#PWR04" H 9550 3400 50  0001 C CNN
+F 1 "GND" H 9555 3477 50  0000 C CNN
+F 2 "" H 9550 3650 50  0001 C CNN
+F 3 "" H 9550 3650 50  0001 C CNN
+	1    9550 3650
+	1    0    0    -1
+$EndComp
+Wire Wire Line
+	9450 3550 9550 3550
+Wire Wire Line
+	9550 3550 9550 3650
+Text GLabel 9550 3250 2    50   Input ~ 10
 SWDIO
-Text GLabel 8200 1300 2    50   Input ~ 10
+Text GLabel 9550 3350 2    50   Input ~ 10
 SWCLK
-Text GLabel 8200 1400 2    50   Input ~ 10
+Text GLabel 9550 3450 2    50   Input ~ 10
 NRST
 Wire Wire Line
-	8100 1200 8200 1200
-Wire Wire Line
-	8100 1300 8200 1300
-Wire Wire Line
-	8100 1400 8200 1400
+	9450 3250 9550 3250
+Wire Wire Line
+	9450 3350 9550 3350
+Wire Wire Line
+	9450 3450 9550 3450
 Text Notes 3600 2850 0    50   ~ 10
-TODO: \n* add PWR_ON signal for the GPS module\n* add pin names/functions
+TODO:\n* add pin names/functions
 $Comp
 L Mainboard-rescue:USBLC6-2SC6-ESD_Protection U2
@@
 Text GLabel 4700 5450 3    50   Input ~ 10
 FM_MOD_SEL
+Wire Wire Line
+	5700 5450 5700 5350
+Text GLabel 5700 5450 3    50   Input ~ 10
+WIFI_EN
+Text Notes 800  5100 0    50   ~ 0
+USART1  GPS\nUSART2  Debug\nUSART3  ESP8266-12\nUSART7  HMI
+Wire Notes Line
+	800  4750 2200 4750
+Wire Notes Line
+	2200 5100 800  5100
+Wire Notes Line
+	2200 4750 2200 5100
+Wire Notes Line
+	800  4750 800  5100
+Wire Wire Line
+	4900 5450 4900 5350
+Wire Wire Line
+	5000 5450 5000 5350
+Text GLabel 4900 5450 3    50   Input ~ 10
+UART7_RX
+Text GLabel 5000 5450 3    50   Input ~ 10
+UART7_TX
+Wire Wire Line
+	5100 5350 5100 5950
+Wire Wire Line
+	5200 5350 5200 5950
 $EndSCHEMATC
