File: kicad/Mainboard/STM32.sch (KiCad schematic (older format))
At the start: 23 parts, among them J1 SWD, J2 USB_OTG, J3 TP1, J4 TP2, U1 STM32F777VIT, U2 USBLC6-2SC6

Commit message: Add files via upload
Connections:
- net WIFI_RST: now reaches U1.44 (P$44)
- no-connect marks 39 -> 38
Other:
- note added: "SPI1 Display\nSPI2 ADF7021 data?"
- note added: "TODO:\n* add pin names/functions\n* connect ADF7021 to STM32"
- note removed: "TODO:\n* add pin names/functions"
- moved on the sheet: Q?, R4, R?
Changed lines of the file:
@@
 NoConn ~ 5400 5350
 NoConn ~ 5500 5350
-NoConn ~ 5600 5350
 Wire Wire Line
 	6900 2350 7000 2350
@@
 L Mainboard-rescue:R_Small-device R4
 U 1 1 5DEC41C2
-P 2450 6400
-F 0 "R4" H 2509 6446 50  0000 L CNN
-F 1 "10k" H 2509 6355 50  0000 L CNN
-F 2 "" H 2450 6400 50  0001 C CNN
-F 3 "~" H 2450 6400 50  0001 C CNN
-	1    2450 6400
-	1    0    0    -1
-$EndComp
-Text GLabel 1900 6600 2    50   Input ~ 10
+P 10150 3250
+F 0 "R4" H 10209 3296 50  0000 L CNN
+F 1 "10k" H 10209 3205 50  0000 L CNN
+F 2 "" H 10150 3250 50  0001 C CNN
+F 3 "~" H 10150 3250 50  0001 C CNN
+	1    10150 3250
+	1    0    0    -1
+$EndComp
+Text GLabel 10050 1450 2    50   Input ~ 10
 BOOT0
 $Comp
 L power:+3V3 #PWR020
 U 1 1 5DEC8A28
-P 2450 6200
-F 0 "#PWR020" H 2450 6050 50  0001 C CNN
-F 1 "+3V3" H 2465 6373 50  0000 C CNN
-F 2 "" H 2450 6200 50  0001 C CNN
-F 3 "" H 2450 6200 50  0001 C CNN
-	1    2450 6200
-	1    0    0    -1
-$EndComp
-Wire Wire Line
-	2450 6200 2450 6300
-Wire Wire Line
-	2450 6500 2450 6600
-Text GLabel 2450 6600 3    50   Input ~ 10
+P 10150 3050
+F 0 "#PWR020" H 10150 2900 50  0001 C CNN
+F 1 "+3V3" H 10165 3223 50  0000 C CNN
+F 2 "" H 10150 3050 50  0001 C CNN
+F 3 "" H 10150 3050 50  0001 C CNN
+	1    10150 3050
+	1    0    0    -1
+$EndComp
+Wire Wire Line
+	10150 3050 10150 3150
+Wire Wire Line
+	10150 3350 10150 3450
+Text GLabel 10150 3450 3    50   Input ~ 10
 NRST
 $Comp
@@
 Wire Wire Line
 	9450 3450 9550 3450
-Text Notes 3600 2850 0    50   ~ 10
-TODO:\n* add pin names/functions
+Text Notes 800  5900 0    50   ~ 0
+TODO:\n* add pin names/functions\n* connect ADF7021 to STM32
 $Comp
 L Mainboard-rescue:USBLC6-2SC6-ESD_Protection U2
@@
 Wire Wire Line
 	6900 2750 7100 2750
-Text GLabel 1300 6900 0    50   Input ~ 10
+Text GLabel 9450 1750 0    50   Input ~ 10
 PTT
 Wire Wire Line
@@
 NoConn ~ 4200 1550
 Wire Wire Line
-	1900 6600 1800 6600
-Wire Wire Line
-	1800 6600 1800 6700
+	10050 1450 9950 1450
+Wire Wire Line
+	9950 1450 9950 1550
 $Comp
 L Device:R_Small R?
 U 1 1 5E0EDCC6
-P 1800 6400
-F 0 "R?" H 1741 6354 50  0000 R CNN
-F 1 "10k" H 1741 6445 50  0000 R CNN
-F 2 "" H 1800 6400 50  0001 C CNN
-F 3 "~" H 1800 6400 50  0001 C CNN
-	1    1800 6400
+P 9950 1250
+F 0 "R?" H 9891 1204 50  0000 R CNN
+F 1 "10k" H 9891 1295 50  0000 R CNN
+F 2 "" H 9950 1250 50  0001 C CNN
+F 3 "~" H 9950 1250 50  0001 C CNN
+	1    9950 1250
 	1    0    0    1
 $EndComp
 Wire Wire Line
-	1800 6500 1800 6600
-Connection ~ 1800 6600
+	9950 1350 9950 1450
+Connection ~ 9950 1450
 $Comp
 L power:+3V3 #PWR?
 U 1 1 5E0F302C
-P 1800 6200
-F 0 "#PWR?" H 1800 6050 50  0001 C CNN
-F 1 "+3V3" H 1815 6373 50  0000 C CNN
-F 2 "" H 1800 6200 50  0001 C CNN
-F 3 "" H 1800 6200 50  0001 C CNN
-	1    1800 6200
-	1    0    0    -1
-$EndComp
-Wire Wire Line
-	1800 6200 1800 6300
+P 9950 1050
+F 0 "#PWR?" H 9950 900 50  0001 C CNN
+F 1 "+3V3" H 9965 1223 50  0000 C CNN
+F 2 "" H 9950 1050 50  0001 C CNN
+F 3 "" H 9950 1050 50  0001 C CNN
+	1    9950 1050
+	1    0    0    -1
+$EndComp
+Wire Wire Line
+	9950 1050 9950 1150
 $Comp
 L power:GND #PWR?
 U 1 1 5E0F8338
-P 1800 7200
-F 0 "#PWR?" H 1800 6950 50  0001 C CNN
-F 1 "GND" H 1805 7027 50  0000 C CNN
-F 2 "" H 1800 7200 50  0001 C CNN
-F 3 "" H 1800 7200 50  0001 C CNN
-	1    1800 7200
-	1    0    0    -1
-$EndComp
-Wire Wire Line
-	1800 7100 1800 7200
+P 9950 2050
+F 0 "#PWR?" H 9950 1800 50  0001 C CNN
+F 1 "GND" H 9955 1877 50  0000 C CNN
+F 2 "" H 9950 2050 50  0001 C CNN
+F 3 "" H 9950 2050 50  0001 C CNN
+	1    9950 2050
+	1    0    0    -1
+$EndComp
+Wire Wire Line
+	9950 1950 9950 2050
 NoConn ~ 4000 1550
 $Comp
 L Transistor_FET:BSS138 Q?
 U 1 1 5E22ECEC
-P 1700 6900
-F 0 "Q?" H 1906 6946 50  0000 L CNN
-F 1 "BSS138" H 1906 6855 50  0000 L CNN
-F 2 "Package_TO_SOT_SMD:SOT-23" H 1900 6825 50  0001 L CIN
-F 3 "https://www.fairchildsemi.com/datasheets/BS/BSS138.pdf" H 1700 6900 50  0001 L CNN
-	1    1700 6900
-	1    0    0    -1
-$EndComp
-Wire Wire Line
-	1500 6900 1300 6900
+P 9850 1750
+F 0 "Q?" H 10056 1796 50  0000 L CNN
+F 1 "BSS138" H 10056 1705 50  0000 L CNN
+F 2 "Package_TO_SOT_SMD:SOT-23" H 10050 1675 50  0001 L CIN
+F 3 "https://www.fairchildsemi.com/datasheets/BS/BSS138.pdf" H 9850 1750 50  0001 L CNN
+	1    9850 1750
+	1    0    0    -1
+$EndComp
+Wire Wire Line
+	9650 1750 9450 1750
 Wire Wire Line
 	4100 5450 4100 5350
@@
 Wire Wire Line
 	5200 5350 5200 5950
+Wire Wire Line
+	5600 5450 5600 5350
+Text GLabel 5600 5450 3    50   Input ~ 10
+WIFI_RST
+Text Notes 800  5450 0    50   ~ 0
+SPI1  Display\nSPI2  ADF7021 data?
+Wire Notes Line
+	800  5300 2200 5300
+Wire Notes Line
+	2200 5450 800  5450
+Wire Notes Line
+	2200 5300 2200 5450
+Wire Notes Line
+	800  5300 800  5450
 $EndSCHEMATC

Commit message: Add files via upload
Connections:
- net ADF_SLE: now reaches U1.56 (P$56)
- net ADF_SDATA: now reaches U1.57 (P$57)
- net ADF_SREAD: now reaches U1.58 (P$58)
- net ADF_SCLK: now reaches U1.59 (P$59)
- net ADF_SWD: now reaches U1.60 (P$60)
- net SPI2_CS renamed ADF_CE
- no-connect marks 38 -> 33
Changed lines of the file:
@@
 BLIGHT_CTRL
 Text GLabel 7100 4250 2    50   Input ~ 10
-SPI2_CS
+ADF_CE
 Text GLabel 7100 4350 2    50   Input ~ 10
 SPI2_MOSI
@@
 	7750 2750 7750 2850
 NoConn ~ 6900 3550
-NoConn ~ 6900 3650
-NoConn ~ 6900 3750
-NoConn ~ 6900 3950
-NoConn ~ 6900 4050
-NoConn ~ 6900 4150
 NoConn ~ 6900 4650
 Text GLabel 6200 1450 1    50   Input ~ 10
@@
 NoConn ~ 6900 3350
 NoConn ~ 6900 3450
-NoConn ~ 6900 3850
 Wire Wire Line
 	4600 5450 4600 5350
@@
 Wire Notes Line
 	800  5300 800  5450
+Text GLabel 7100 4150 2    50   Input ~ 10
+ADF_SLE
+Text GLabel 7100 4050 2    50   Input ~ 10
+ADF_SDATA
+Text GLabel 7100 3950 2    50   Input ~ 10
+ADF_SREAD
+Text GLabel 7100 3850 2    50   Input ~ 10
+ADF_SCLK
+Text GLabel 7100 3750 2    50   Input ~ 10
+ADF_SWD
+NoConn ~ 6900 3650
+Wire Wire Line
+	6900 3750 7100 3750
+Wire Wire Line
+	7100 3850 6900 3850
+Wire Wire Line
+	6900 3950 7100 3950
+Wire Wire Line
+	6900 4050 7100 4050
+Wire Wire Line
+	7100 4150 6900 4150
 $EndSCHEMATC
