File: kicad/Mainboard/STM32.sch (KiCad schematic (older format))
At the start: 23 parts, among them J1 SWD, J2 USB_OTG, J3 TP1, J4 TP2, U1 STM32F777VIT, U2 USBLC6-2SC6

Commit message: Annotated parts, again.
Parts:
- gave numbers to parts that had none: 2
- renumbered C7 to C3, C3 to C4, C4 to C5, C5 to C6, C6 to C7, J3 to J1, J4 to J2, J2 to J3, J1 to J4, R4 to R3, R2 to R4, R3 to R5

Commit message: Started assigning footprints
Parts:
- C1, C2, C3, C4, C5, C6, C7: footprint (none) -> Capacitor_SMD:C_0603_1608Metric
- FB1, FB2: footprint (none) -> Inductor_SMD:L_0603_1608Metric
- Q1: symbol Transistor_FET:BSS138 -> Mainboard-rescue:BSS138-Transistor_FET
- R2: symbol Device:R_Small -> Mainboard-rescue:R_Small-Device
Other:
- note added: "TODO:\n* add pin names/functions"
- note removed: "TODO:\n* add pin names/functions\n* connect ADF7021 to STM32"
Changed lines of the file:
@@
 F 0 "FB1" V 963 1150 50  0000 C CNN
 F 1 "TBD" V 1054 1150 50  0000 C CNN
-F 2 "" V 1130 1150 50  0001 C CNN
+F 2 "Inductor_SMD:L_0603_1608Metric" V 1130 1150 50  0001 C CNN
 F 3 "~" H 1200 1150 50  0001 C CNN
 	1    1200 1150
@@
 F 0 "FB2" V 963 1550 50  0000 C CNN
 F 1 "TBD" V 1054 1550 50  0000 C CNN
-F 2 "" V 1130 1550 50  0001 C CNN
+F 2 "Inductor_SMD:L_0603_1608Metric" V 1130 1550 50  0001 C CNN
 F 3 "~" H 1200 1550 50  0001 C CNN
 	1    1200 1550
@@
 F 0 "C1" H 1492 1796 50  0000 L CNN
 F 1 "100n" H 1492 1705 50  0000 L CNN
-F 2 "" H 1400 1750 50  0001 C CNN
+F 2 "Capacitor_SMD:C_0603_1608Metric" H 1400 1750 50  0001 C CNN
 F 3 "~" H 1400 1750 50  0001 C CNN
 	1    1400 1750
@@
 F 0 "C2" H 1892 1796 50  0000 L CNN
 F 1 "100n" H 1892 1705 50  0000 L CNN
-F 2 "" H 1800 1750 50  0001 C CNN
+F 2 "Capacitor_SMD:C_0603_1608Metric" H 1800 1750 50  0001 C CNN
 F 3 "~" H 1800 1750 50  0001 C CNN
 	1    1800 1750
@@
 F 0 "C3" H 5908 6004 50  0000 R CNN
 F 1 "2u2" H 5908 6095 50  0000 R CNN
-F 2 "" H 6000 6050 50  0001 C CNN
+F 2 "Capacitor_SMD:C_0603_1608Metric" H 6000 6050 50  0001 C CNN
 F 3 "~" H 6000 6050 50  0001 C CNN
 	1    6000 6050
@@
 F 0 "C4" H 7658 2604 50  0000 R CNN
 F 1 "2u2" H 7658 2695 50  0000 R CNN
-F 2 "" H 7750 2650 50  0001 C CNN
+F 2 "Capacitor_SMD:C_0603_1608Metric" H 7750 2650 50  0001 C CNN
 F 3 "~" H 7750 2650 50  0001 C CNN
 	1    7750 2650
@@
 	9450 3450 9550 3450
 Text Notes 800  5900 0    50   ~ 0
-TODO:\n* add pin names/functions\n* connect ADF7021 to STM32
+TODO:\n* add pin names/functions
 $Comp
 L Mainboard-rescue:USBLC6-2SC6-ESD_Protection U2
@@
 F 0 "C5" H 8458 5654 50  0000 R CNN
 F 1 "10n" H 8458 5745 50  0000 R CNN
-F 2 "" H 8550 5700 50  0001 C CNN
+F 2 "Capacitor_SMD:C_0603_1608Metric" H 8550 5700 50  0001 C CNN
 F 3 "~" H 8550 5700 50  0001 C CNN
 	1    8550 5700
@@
 F 0 "C6" H 10058 5854 50  0000 R CNN
 F 1 "47p" H 10058 5945 50  0000 R CNN
-F 2 "" H 10150 5900 50  0001 C CNN
+F 2 "Capacitor_SMD:C_0603_1608Metric" H 10150 5900 50  0001 C CNN
 F 3 "~" H 10150 5900 50  0001 C CNN
 	1    10150 5900
@@
 F 0 "C7" H 10258 5854 50  0000 R CNN
 F 1 "47p" H 10258 5945 50  0000 R CNN
-F 2 "" H 10350 5900 50  0001 C CNN
+F 2 "Capacitor_SMD:C_0603_1608Metric" H 10350 5900 50  0001 C CNN
 F 3 "~" H 10350 5900 50  0001 C CNN
 	1    10350 5900
@@
 	9950 1450 9950 1550
 $Comp
-L Device:R_Small R2
+L Mainboard-rescue:R_Small-Device R2
 U 1 1 5E0EDCC6
 P 9950 1250
@@
 NoConn ~ 4000 1550
 $Comp
-L Transistor_FET:BSS138 Q1
+L Mainboard-rescue:BSS138-Transistor_FET Q1
 U 1 1 5E22ECEC
 P 9850 1750

Commit message: Add files via upload
assigned some more footprints
Parts:
- J1, J2: footprint (none) -> TestPoint:TestPoint_Pad_D1.0mm
- L1: footprint (none) -> Inductor_SMD:L_0603_1608Metric
- R1, R2, R3, R4, R5: footprint (none) -> Resistor_SMD:R_0603_1608Metric
- U1: footprint (none) -> Package_QFP:LQFP-100_14x14mm_P0.5mm
Other:
- note removed: "TODO:\n* add pin names/functions"
Changed lines of the file:
@@
 F 0 "U1" H 4950 3550 59  0000 L CNN
 F 1 "STM32F777VIT" H 4700 3400 59  0000 L CNN
-F 2 "" H 5000 3450 50  0001 C CNN
+F 2 "Package_QFP:LQFP-100_14x14mm_P0.5mm" H 5000 3450 50  0001 C CNN
 F 3 "" H 5000 3450 50  0001 C CNN
 	1    5000 3450
@@
 F 0 "J1" V 5200 6100 50  0000 R CNN
 F 1 "TP1" V 5200 6250 50  0000 R CNN
-F 2 "" H 5300 5950 50  0001 C CNN
+F 2 "TestPoint:TestPoint_Pad_D1.0mm" H 5300 5950 50  0001 C CNN
 F 3 "" H 5300 5950 50  0001 C CNN
 	1    5100 5950
@@
 F 0 "J2" V 5300 6100 50  0000 R CNN
 F 1 "TP2" V 5300 6250 50  0000 R CNN
-F 2 "" H 5400 5950 50  0001 C CNN
+F 2 "TestPoint:TestPoint_Pad_D1.0mm" H 5400 5950 50  0001 C CNN
 F 3 "" H 5400 5950 50  0001 C CNN
 	1    5200 5950
@@
 F 0 "R3" H 10209 3296 50  0000 L CNN
 F 1 "10k" H 10209 3205 50  0000 L CNN
-F 2 "" H 10150 3250 50  0001 C CNN
+F 2 "Resistor_SMD:R_0603_1608Metric" H 10150 3250 50  0001 C CNN
 F 3 "~" H 10150 3250 50  0001 C CNN
 	1    10150 3250
@@
 Wire Wire Line
 	9450 3450 9550 3450
-Text Notes 800  5900 0    50   ~ 0
-TODO:\n* add pin names/functions
 $Comp
 L Mainboard-rescue:USBLC6-2SC6-ESD_Protection U2
@@
 F 0 "L1" V 8500 4850 50  0000 L CNN
 F 1 "100MHz" V 8650 4750 50  0000 L CNN
-F 2 "" H 8550 4900 50  0001 C CNN
+F 2 "Inductor_SMD:L_0603_1608Metric" H 8550 4900 50  0001 C CNN
 F 3 "~" H 8550 4900 50  0001 C CNN
 	1    8550 4900
@@
 F 0 "R1" H 8859 4946 50  0000 L CNN
 F 1 "1k5" H 8859 4855 50  0000 L CNN
-F 2 "" H 8800 4900 50  0001 C CNN
+F 2 "Resistor_SMD:R_0603_1608Metric" H 8800 4900 50  0001 C CNN
 F 3 "~" H 8800 4900 50  0001 C CNN
 	1    8800 4900
@@
 F 0 "R4" V 10354 5300 50  0000 C CNN
 F 1 "27" V 10445 5300 50  0000 C CNN
-F 2 "" H 10550 5300 50  0001 C CNN
+F 2 "Resistor_SMD:R_0603_1608Metric" H 10550 5300 50  0001 C CNN
 F 3 "~" H 10550 5300 50  0001 C CNN
 	1    10550 5300
@@
 F 0 "R5" V 10354 5700 50  0000 C CNN
 F 1 "27" V 10445 5700 50  0000 C CNN
-F 2 "" H 10550 5700 50  0001 C CNN
+F 2 "Resistor_SMD:R_0603_1608Metric" H 10550 5700 50  0001 C CNN
 F 3 "~" H 10550 5700 50  0001 C CNN
 	1    10550 5700
@@
 F 0 "R2" H 9891 1204 50  0000 R CNN
 F 1 "10k" H 9891 1295 50  0000 R CNN
-F 2 "" H 9950 1250 50  0001 C CNN
+F 2 "Resistor_SMD:R_0603_1608Metric" H 9950 1250 50  0001 C CNN
 F 3 "~" H 9950 1250 50  0001 C CNN
 	1    9950 1250

Commit message: - Added footprint library - TR-9 - Imported a few footprints - Designed a MicroSD card slot footprint - Assignment footprints to corresponding elements on schematic
Parts:
- OS1: footprint (none) -> TR-9:ECS-3225-MV-160-CN-TR
Changed lines of the file:
@@
 EESchema Schematic File Version 4
-LIBS:Mainboard-cache
 EELAYER 30 0
 EELAYER END
@@
 F 0 "OS1" H 1350 3700 59  0000 C CNN
 F 1 "ECS-3225MV-160-CN-TR" H 1850 3000 59  0000 C CNN
-F 2 "" H 1550 3350 50  0001 C CNN
+F 2 "TR-9:ECS-3225-MV-160-CN-TR" H 1550 3350 50  0001 C CNN
 F 3 "" H 1550 3350 50  0001 C CNN
 	1    1550 3350

Commit message: Assigned SMA as antenna connector
Parts:
- J3: footprint (none) -> Connector_USB:USB_Mini-B_Wuerth_65100516121_Horizontal
Changed lines of the file:
@@
 F 0 "J3" H 8207 5767 50  0000 C CNN
 F 1 "USB_OTG" H 8207 5676 50  0000 C CNN
-F 2 "" H 8300 5250 50  0001 C CNN
+F 2 "Connector_USB:USB_Mini-B_Wuerth_65100516121_Horizontal" H 8300 5250 50  0001 C CNN
 F 3 "" H 8300 5250 50  0001 C CNN
 	1    8150 5300

Commit message: - designed and added footprint for L8 RF inductor
Parts:
- J4: footprint (none) -> Connector_PinHeader_2.54mm:PinHeader_1x05_P2.54mm_Vertical
Changed lines of the file:
@@
 F 0 "J4" H 9168 2925 50  0000 C CNN
 F 1 "SWD" H 9168 3016 50  0000 C CNN
-F 2 "" H 9250 3350 50  0001 C CNN
+F 2 "Connector_PinHeader_2.54mm:PinHeader_1x05_P2.54mm_Vertical" H 9250 3350 50  0001 C CNN
 F 3 "~" H 9250 3350 50  0001 C CNN
 	1    9250 3350

Commit message: Added HMC RF switch Corrected SOIC footprints assignment
Parts:
- U2: footprint TO_SOT_Packages_SMD:SOT-23-6 -> Package_TO_SOT_SMD:SOT-23-6
Changed lines of the file:
@@
 F 0 "U2" H 9400 5967 50  0000 C CNN
 F 1 "USBLC6-2SC6" H 9400 5876 50  0000 C CNN
-F 2 "TO_SOT_Packages_SMD:SOT-23-6" H 10050 5850 50  0001 C CNN
+F 2 "Package_TO_SOT_SMD:SOT-23-6" H 10050 5850 50  0001 C CNN
 F 3 "http://www2.st.com/resource/en/datasheet/CD00050750.pdf" H 9150 5850 50  0001 C CNN
 	1    9400 5500
