File: kicad/Mainboard/PSU.sch (KiCad schematic (older format))
At the start: 24 parts, among them J5 BATT, U3 LD1117S50TR_SOT223, U4 LD1117S33TR_SOT223

Commit message: Add files via upload
Other:
- moved on the sheet: D1, F1, J5
Changed lines of the file:
@@
 L Mainboard-rescue:Conn_01x03-conn J5
 U 1 1 5DEDCC67
-P 1550 1650
-F 0 "J5" H 1468 1967 50  0000 C CNN
-F 1 "BATT" H 1468 1876 50  0000 C CNN
-F 2 "" H 1550 1650 50  0001 C CNN
-F 3 "~" H 1550 1650 50  0001 C CNN
-	1    1550 1650
+P 1500 3600
+F 0 "J5" H 1418 3917 50  0000 C CNN
+F 1 "BATT" H 1418 3826 50  0000 C CNN
+F 2 "" H 1500 3600 50  0001 C CNN
+F 3 "~" H 1500 3600 50  0001 C CNN
+	1    1500 3600
 	-1   0    0    -1
 $EndComp
@@
 L Mainboard-rescue:Fuse_Small-device F1
 U 1 1 5DEDD25C
-P 1950 1550
-F 0 "F1" H 1950 1735 50  0000 C CNN
-F 1 "2A" H 1950 1644 50  0000 C CNN
-F 2 "" H 1950 1550 50  0001 C CNN
-F 3 "~" H 1950 1550 50  0001 C CNN
-	1    1950 1550
+P 1900 3500
+F 0 "F1" H 1900 3685 50  0000 C CNN
+F 1 "2A" H 1900 3594 50  0000 C CNN
+F 2 "" H 1900 3500 50  0001 C CNN
+F 3 "~" H 1900 3500 50  0001 C CNN
+	1    1900 3500
 	1    0    0    -1
 $EndComp
 Wire Wire Line
-	1750 1550 1850 1550
-NoConn ~ 1750 1650
+	1700 3500 1800 3500
+NoConn ~ 1700 3600
 $Comp
 L power:+BATT #PWR029
 U 1 1 5DEDD9E9
-P 2150 1450
-F 0 "#PWR029" H 2150 1300 50  0001 C CNN
-F 1 "+BATT" H 2165 1623 50  0000 C CNN
-F 2 "" H 2150 1450 50  0001 C CNN
-F 3 "" H 2150 1450 50  0001 C CNN
-	1    2150 1450
+P 2100 3400
+F 0 "#PWR029" H 2100 3250 50  0001 C CNN
+F 1 "+BATT" H 2115 3573 50  0000 C CNN
+F 2 "" H 2100 3400 50  0001 C CNN
+F 3 "" H 2100 3400 50  0001 C CNN
+	1    2100 3400
 	1    0    0    -1
 $EndComp
 Wire Wire Line
-	2050 1550 2150 1550
+	2000 3500 2100 3500
 Wire Wire Line
-	2150 1550 2150 1450
+	2100 3500 2100 3400
 $Comp
 L Mainboard-rescue:D_Small-device D1
 U 1 1 5DEDE398
-P 2150 1750
-F 0 "D1" V 2104 1818 50  0000 L CNN
-F 1 "CGRM4007-G" V 2195 1818 50  0000 L CNN
-F 2 "" V 2150 1750 50  0001 C CNN
-F 3 "~" V 2150 1750 50  0001 C CNN
-	1    2150 1750
+P 2100 3700
+F 0 "D1" V 2054 3768 50  0000 L CNN
+F 1 "CGRM4007-G" V 2145 3768 50  0000 L CNN
+F 2 "" V 2100 3700 50  0001 C CNN
+F 3 "~" V 2100 3700 50  0001 C CNN
+	1    2100 3700
 	0    1    1    0
 $EndComp
 Wire Wire Line
-	2150 1550 2150 1650
-Connection ~ 2150 1550
+	2100 3500 2100 3600
+Connection ~ 2100 3500
 $Comp
 L power:GND #PWR031
 U 1 1 5DEDEF0C
-P 2150 1950
-F 0 "#PWR031" H 2150 1700 50  0001 C CNN
-F 1 "GND" H 2155 1777 50  0000 C CNN
-F 2 "" H 2150 1950 50  0001 C CNN
-F 3 "" H 2150 1950 50  0001 C CNN
-	1    2150 1950
+P 2100 3900
+F 0 "#PWR031" H 2100 3650 50  0001 C CNN
+F 1 "GND" H 2105 3727 50  0000 C CNN
+F 2 "" H 2100 3900 50  0001 C CNN
+F 3 "" H 2100 3900 50  0001 C CNN
+	1    2100 3900
 	1    0    0    -1
 $EndComp
@@
 L power:GND #PWR030
 U 1 1 5DEDF112
-P 1850 1950
-F 0 "#PWR030" H 1850 1700 50  0001 C CNN
-F 1 "GND" H 1855 1777 50  0000 C CNN
-F 2 "" H 1850 1950 50  0001 C CNN
-F 3 "" H 1850 1950 50  0001 C CNN
-	1    1850 1950
+P 1800 3900
+F 0 "#PWR030" H 1800 3650 50  0001 C CNN
+F 1 "GND" H 1805 3727 50  0000 C CNN
+F 2 "" H 1800 3900 50  0001 C CNN
+F 3 "" H 1800 3900 50  0001 C CNN
+	1    1800 3900
 	1    0    0    -1
 $EndComp
 Wire Wire Line
-	1750 1750 1850 1750
+	1700 3700 1800 3700
 Wire Wire Line
-	1850 1750 1850 1950
+	1800 3700 1800 3900
 Wire Wire Line
-	2150 1850 2150 1950
+	2100 3800 2100 3900
 $Comp
 L Mainboard-rescue:LD1117S33TR_SOT223-regul U4

Commit message: Add files via upload
Parts:
- added J?: POT_PWR_SW, symbol Connector_Generic:Conn_01x02
Connections:
- net +BATT: now also J?.2 (Pin_2); no longer D1.1 (K), F1.2
- new net: D1.1 (K), F1.2, J?.1 (Pin_1)
Changed lines of the file:
@@
 L power:+BATT #PWR029
 U 1 1 5DEDD9E9
-P 2100 3400
-F 0 "#PWR029" H 2100 3250 50  0001 C CNN
-F 1 "+BATT" H 2115 3573 50  0000 C CNN
-F 2 "" H 2100 3400 50  0001 C CNN
-F 3 "" H 2100 3400 50  0001 C CNN
-	1    2100 3400
-	1    0    0    -1
+P 2500 3500
+F 0 "#PWR029" H 2500 3350 50  0001 C CNN
+F 1 "+BATT" H 2515 3673 50  0000 C CNN
+F 2 "" H 2500 3500 50  0001 C CNN
+F 3 "" H 2500 3500 50  0001 C CNN
+	1    2500 3500
+	0    1    1    0
 $EndComp
 Wire Wire Line
 	2000 3500 2100 3500
-Wire Wire Line
-	2100 3500 2100 3400
 $Comp
 L Mainboard-rescue:D_Small-device D1
@@
 Wire Wire Line
 	2100 3500 2100 3600
-Connection ~ 2100 3500
 $Comp
 L power:GND #PWR031
@@
 Wire Notes Line
 	6250 2700 3100 2700
+$Comp
+L Connector_Generic:Conn_01x02 J?
+U 1 1 5E2A6BF0
+P 2250 3250
+F 0 "J?" V 2214 3062 50  0000 R CNN
+F 1 "POT_PWR_SW" V 2123 3062 50  0000 R CNN
+F 2 "" H 2250 3250 50  0001 C CNN
+F 3 "~" H 2250 3250 50  0001 C CNN
+	1    2250 3250
+	0    -1   -1   0
+$EndComp
+Wire Wire Line
+	2100 3500 2250 3500
+Wire Wire Line
+	2250 3500 2250 3450
+Connection ~ 2100 3500
+Wire Wire Line
+	2350 3500 2350 3450
+Wire Wire Line
+	2350 3500 2500 3500
 $EndSCHEMATC

Commit message: Annotated parts, again.
Parts:
- gave numbers to parts that had none: 1
- renumbered C13 to C10, C8 to C11, C15 to C12, C9 to C13, C16 to C14, C10 to C15, C17 to C16, C11 to C17, C12 to C8, C14 to C9, R5 to R6, R6 to R7
Changed lines of the file:
@@
 EESchema Schematic File Version 4
-LIBS:Mainboard-cache
 EELAYER 30 0
 EELAYER END
@@
 NoConn ~ 1700 3600
 $Comp
-L power:+BATT #PWR029
+L power:+BATT #PWR037
 U 1 1 5DEDD9E9
 P 2500 3500
-F 0 "#PWR029" H 2500 3350 50  0001 C CNN
+F 0 "#PWR037" H 2500 3350 50  0001 C CNN
 F 1 "+BATT" H 2515 3673 50  0000 C CNN
 F 2 "" H 2500 3500 50  0001 C CNN
@@
 	2100 3500 2100 3600
 $Comp
-L power:GND #PWR031
+L power:GND #PWR035
 U 1 1 5DEDEF0C
 P 2100 3900
-F 0 "#PWR031" H 2100 3650 50  0001 C CNN
+F 0 "#PWR035" H 2100 3650 50  0001 C CNN
 F 1 "GND" H 2105 3727 50  0000 C CNN
 F 2 "" H 2100 3900 50  0001 C CNN
@@
 $EndComp
 $Comp
-L power:GND #PWR030
+L power:GND #PWR033
 U 1 1 5DEDF112
 P 1800 3900
-F 0 "#PWR030" H 1800 3650 50  0001 C CNN
+F 0 "#PWR033" H 1800 3650 50  0001 C CNN
 F 1 "GND" H 1805 3727 50  0000 C CNN
 F 2 "" H 1800 3900 50  0001 C CNN
@@
 $EndComp
 $Comp
-L power:+3V3 #PWR036
+L power:+3V3 #PWR046
 U 1 1 5DEDFD78
 P 6000 3000
-F 0 "#PWR036" H 6000 2850 50  0001 C CNN
+F 0 "#PWR046" H 6000 2850 50  0001 C CNN
 F 1 "+3V3" H 6015 3173 50  0000 C CNN
 F 2 "" H 6000 3000 50  0001 C CNN
@@
 	6000 3100 6000 3000
 $Comp
-L power:+BATT #PWR034
+L power:+BATT #PWR040
 U 1 1 5DEE07CE
 P 3850 3000
-F 0 "#PWR034" H 3850 2850 50  0001 C CNN
+F 0 "#PWR040" H 3850 2850 50  0001 C CNN
 F 1 "+BATT" H 3865 3173 50  0000 C CNN
 F 2 "" H 3850 3000 50  0001 C CNN
@@
 	3850 3100 4150 3100
 $Comp
-L Mainboard-rescue:CP_Small-device C12
+L Mainboard-rescue:CP_Small-device C8
 U 1 1 5DEE1557
 P 3550 3100
-F 0 "C12" V 3325 3100 50  0000 C CNN
+F 0 "C8" V 3325 3100 50  0000 C CNN
 F 1 "22u/TA" V 3416 3100 50  0000 C CNN
 F 2 "" H 3550 3100 50  0001 C CNN
@@
 	3350 3100 3350 3200
 $Comp
-L power:GND #PWR037
+L power:GND #PWR038
 U 1 1 5DEE30CD
 P 3350 3200
-F 0 "#PWR037" H 3350 2950 50  0001 C CNN
+F 0 "#PWR038" H 3350 2950 50  0001 C CNN
 F 1 "GND" H 3355 3027 50  0000 C CNN
 F 2 "" H 3350 3200 50  0001 C CNN
@@
 $EndComp
 $Comp
-L Mainboard-rescue:R_Small-device R5
+L Mainboard-rescue:R_Small-device R6
 U 1 1 5DEE367B
 P 3850 3300
-F 0 "R5" H 3909 3346 50  0000 L CNN
+F 0 "R6" H 3909 3346 50  0000 L CNN
 F 1 "9k1" H 3909 3255 50  0000 L CNN
 F 2 "" H 3850 3300 50  0001 C CNN
@@
 $EndComp
 $Comp
-L Mainboard-rescue:R_Small-device R6
+L Mainboard-rescue:R_Small-device R7
 U 1 1 5DEE3FDD
 P 3850 3700
-F 0 "R6" H 3909 3746 50  0000 L CNN
+F 0 "R7" H 3909 3746 50  0000 L CNN
 F 1 "1k" H 3909 3655 50  0000 L CNN
 F 2 "" H 3850 3700 50  0001 C CNN
@@
 	3850 3400 3850 3500
 $Comp
-L power:GND #PWR040
+L power:GND #PWR041
 U 1 1 5DEE4B50
 P 3850 3900
-F 0 "#PWR040" H 3850 3650 50  0001 C CNN
+F 0 "#PWR041" H 3850 3650 50  0001 C CNN
 F 1 "GND" H 3855 3727 50  0000 C CNN
 F 2 "" H 3850 3900 50  0001 C CNN
@@
 	3850 3800 3850 3900
 $Comp
-L Mainboard-rescue:C_Small-device C14
+L Mainboard-rescue:C_Small-device C9
 U 1 1 5DEE5372
 P 3600 3700
-F 0 "C14" H 3508 3654 50  0000 R CNN
+F 0 "C9" H 3508 3654 50  0000 R CNN
 F 1 "10n" H 3508 3745 50  0000 R CNN
 F 2 "" H 3600 3700 50  0001 C CNN
@@
 ADC2_3
 $Comp
-L power:GND #PWR043
+L power:GND #PWR045
 U 1 1 5DEE6C72
 P 5450 3900
-F 0 "#PWR043" H 5450 3650 50  0001 C CNN
+F 0 "#PWR045" H 5450 3650 50  0001 C CNN
 F 1 "GND" H 5455 3727 50  0000 C CNN
 F 2 "" H 5450 3900 50  0001 C CNN
@@
 $EndComp
 $Comp
-L power:GND #PWR045
+L power:GND #PWR031
 U 1 1 5DEECC7E
 P 1450 6800
-F 0 "#PWR045" H 1450 6550 50  0001 C CNN
+F 0 "#PWR031" H 1450 6550 50  0001 C CNN
 F 1 "GND" H 1455 6627 50  0000 C CNN
 F 2 "" H 1450 6800 50  0001 C CNN
@@
 $EndComp
 $Comp
-L power:GND #PWR046
+L power:GND #PWR032
 U 1 1 5DEED1C2
 P 1700 6800
-F 0 "#PWR046" H 1700 6550 50  0001 C CNN
+F 0 "#PWR032" H 1700 6550 50  0001 C CNN
 F 1 "GND" H 1705 6627 50  0000 C CNN
 F 2 "" H 1700 6800 50  0001 C CNN
@@
 $EndComp
 $Comp
-L power:GND #PWR047
+L power:GND #PWR034
 U 1 1 5DEED3FC
 P 1950 6800
-F 0 "#PWR047" H 1950 6550 50  0001 C CNN
+F 0 "#PWR034" H 1950 6550 50  0001 C CNN
 F 1 "GND" H 1955 6627 50  0000 C CNN
 F 2 "" H 1950 6800 50  0001 C CNN
@@
 $EndComp
 $Comp
-L power:GND #PWR048
+L power:GND #PWR036
 U 1 1 5DEED62E
 P 2200 6800
-F 0 "#PWR048" H 2200 6550 50  0001 C CNN
+F 0 "#PWR036" H 2200 6550 50  0001 C CNN
 F 1 "GND" H 2205 6627 50  0000 C CNN
 F 2 "" H 2200 6800 50  0001 C CNN
@@
 	1450 6700 1450 6800
 $Comp
-L Mainboard-rescue:C_Small-device C8
+L Mainboard-rescue:C_Small-device C11
 U 1 1 5DEF07B1
 P 7650 2500
-F 0 "C8" H 7742 2546 50  0000 L CNN
+F 0 "C11" H 7742 2546 50  0000 L CNN
 F 1 "22u/TA" H 7742 2455 50  0000 L CNN
 F 2 "" H 7650 2500 50  0001 C CNN
@@
 $EndComp
 $Comp
-L Mainboard-rescue:C_Small-device C9
+L Mainboard-rescue:C_Small-device C13
 U 1 1 5DEF09D7
 P 8150 2500
-F 0 "C9" H 8242 2546 50  0000 L CNN
+F 0 "C13" H 8242 2546 50  0000 L CNN
 F 1 "22u/TA" H 8242 2455 50  0000 L CNN
 F 2 "" H 8150 2500 50  0001 C CNN
@@
 $EndComp
 $Comp
-L Mainboard-rescue:C_Small-device C10
+L Mainboard-rescue:C_Small-device C15
 U 1 1 5DEF0D8F
 P 8650 2500
-F 0 "C10" H 8742 2546 50  0000 L CNN
+F 0 "C15" H 8742 2546 50  0000 L CNN
 F 1 "22u/TA" H 8742 2455 50  0000 L CNN
 F 2 "" H 8650 2500 50  0001 C CNN
@@
 $EndComp
 $Comp
-L Mainboard-rescue:C_Small-device C11
+L Mainboard-rescue:C_Small-device C17
 U 1 1 5DEF110B
 P 9150 2500
-F 0 "C11" H 9242 2546 50  0000 L CNN
+F 0 "C17" H 9242 2546 50  0000 L CNN
 F 1 "22u/TA" H 9242 2455 50  0000 L CNN
 F 2 "" H 9150 2500 50  0001 C CNN
@@
 $EndComp
 $Comp
-L power:+3V3 #PWR032
+L power:+3V3 #PWR047
 U 1 1 5DEF13D8
 P 7650 2200
-F 0 "#PWR032" H 7650 2050 50  0001 C CNN
+F 0 "#PWR047" H 7650 2050 50  0001 C CNN
 F 1 "+3V3" H 7665 2373 50  0000 C CNN
 F 2 "" H 7650 2200 50  0001 C CNN
@@
 Connection ~ 8650 2300
 $Comp
-L power:GND #PWR033
+L power:GND #PWR048
 U 1 1 5DEF35A4
 P 7650 2800
-F 0 "#PWR033" H 7650 2550 50  0001 C CNN
+F 0 "#PWR048" H 7650 2550 50  0001 C CNN
 F 1 "GND" H 7655 2627 50  0000 C CNN
 F 2 "" H 7650 2800 50  0001 C CNN
@@
 STM32
 $Comp
-L Mainboard-rescue:C_Small-device C15
+L Mainboard-rescue:C_Small-device C12
 U 1 1 5DEF7F00
 P 7650 3950
-F 0 "C15" H 7742 3996 50  0000 L CNN
+F 0 "C12" H 7742 3996 50  0000 L CNN
 F 1 "22u/TA" H 7742 3905 50  0000 L CNN
 F 2 "" H 7650 3950 50  0001 C CNN
@@
 $EndComp
 $Comp
-L Mainboard-rescue:C_Small-device C16
+L Mainboard-rescue:C_Small-device C14
 U 1 1 5DEF7F0A
 P 8150 3950
-F 0 "C16" H 8242 3996 50  0000 L CNN
+F 0 "C14" H 8242 3996 50  0000 L CNN
 F 1 "22u/TA" H 8242 3905 50  0000 L CNN
 F 2 "" H 8150 3950 50  0001 C CNN
@@
 $EndComp
 $Comp
-L Mainboard-rescue:C_Small-device C17
+L Mainboard-rescue:C_Small-device C16
 U 1 1 5DEF7F14
 P 8650 3950
-F 0 "C17" H 8742 3996 50  0000 L CNN
+F 0 "C16" H 8742 3996 50  0000 L CNN
 F 1 "22u/TA" H 8742 3905 50  0000 L CNN
 F 2 "" H 8650 3950 50  0001 C CNN
@@
 Connection ~ 9150 4150
 $Comp
-L power:+3V3 #PWR038
+L power:+3V3 #PWR049
 U 1 1 5DF0772F
 P 7650 3650
-F 0 "#PWR038" H 7650 3500 50  0001 C CNN
+F 0 "#PWR049" H 7650 3500 50  0001 C CNN
 F 1 "+3V3" H 7665 3823 50  0000 C CNN
 F 2 "" H 7650 3650 50  0001 C CNN
@@
 Connection ~ 7650 3750
 $Comp
-L power:GND #PWR044
+L power:GND #PWR050
 U 1 1 5DF08D83
 P 7650 4250
-F 0 "#PWR044" H 7650 4000 50  0001 C CNN
+F 0 "#PWR050" H 7650 4000 50  0001 C CNN
 F 1 "GND" H 7655 4077 50  0000 C CNN
 F 2 "" H 7650 4250 50  0001 C CNN
@@
 $EndComp
 $Comp
-L Mainboard-rescue:C_Small-device C13
+L Mainboard-rescue:C_Small-device C10
 U 1 1 5DFAF77C
 P 4950 3600
-F 0 "C13" H 5042 3646 50  0000 L CNN
+F 0 "C10" H 5042 3646 50  0000 L CNN
 F 1 "100n" H 5042 3555 50  0000 L CNN
 F 2 "" H 4950 3600 50  0001 C CNN
@@
 	4950 3100 5150 3100
 $Comp
-L power:GND #PWR042
+L power:GND #PWR044
 U 1 1 5DFBA5D8
 P 4950 3900
-F 0 "#PWR042" H 4950 3650 50  0001 C CNN
+F 0 "#PWR044" H 4950 3650 50  0001 C CNN
 F 1 "GND" H 4955 3727 50  0000 C CNN
 F 2 "" H 4950 3900 50  0001 C CNN
@@
 $EndComp
 $Comp
-L power:GND #PWR041
+L power:GND #PWR042
 U 1 1 5DFBA860
 P 4450 3900
-F 0 "#PWR041" H 4450 3650 50  0001 C CNN
+F 0 "#PWR042" H 4450 3650 50  0001 C CNN
 F 1 "GND" H 4455 3727 50  0000 C CNN
 F 2 "" H 4450 3900 50  0001 C CNN
@@
 	4950 3100 4950 3000
 $Comp
-L power:+5V #PWR035
+L power:+5V #PWR043
 U 1 1 5DFBF386
 P 4950 3000
-F 0 "#PWR035" H 4950 2850 50  0001 C CNN
+F 0 "#PWR043" H 4950 2850 50  0001 C CNN
 F 1 "+5V" H 4965 3173 50  0000 C CNN
 F 2 "" H 4950 3000 50  0001 C CNN
@@
 	6250 2700 3100 2700
 $Comp
-L Connector_Generic:Conn_01x02 J?
+L Connector_Generic:Conn_01x02 J6
 U 1 1 5E2A6BF0
 P 2250 3250
-F 0 "J?" V 2214 3062 50  0000 R CNN
+F 0 "J6" V 2214 3062 50  0000 R CNN
 F 1 "POT_PWR_SW" V 2123 3062 50  0000 R CNN
 F 2 "" H 2250 3250 50  0001 C CNN

Commit message: Started assigning footprints
Parts:
- C10, C18, C19, C20, C9: footprint (none) -> Capacitor_SMD:C_0603_1608Metric
- C11, C12, C13, C14, C15, C16, C17, C8: footprint (none) -> Capacitor_Tantalum_SMD:CP_EIA-3216-18_Kemet-A; Partno (none) -> TAJA226K006RNJV
- D1: footprint (none) -> Diode_SMD:D_SOD-123
- F1: footprint (none) -> Fuse:Fuse_1812_4532Metric
- H1, H2, H3, H4: footprint (none) -> Mounting_Holes:MountingHole_2.2mm_M2_ISO14580_Pad
- J6: symbol Connector_Generic:Conn_01x02 -> Mainboard-rescue:Conn_01x02-Connector_Generic
Changed lines of the file:
@@
 F 0 "F1" H 1900 3685 50  0000 C CNN
 F 1 "2A" H 1900 3594 50  0000 C CNN
-F 2 "" H 1900 3500 50  0001 C CNN
+F 2 "Fuse:Fuse_1812_4532Metric" H 1900 3500 50  0001 C CNN
 F 3 "~" H 1900 3500 50  0001 C CNN
 	1    1900 3500
@@
 F 0 "D1" V 2054 3768 50  0000 L CNN
 F 1 "CGRM4007-G" V 2145 3768 50  0000 L CNN
-F 2 "" V 2100 3700 50  0001 C CNN
+F 2 "Diode_SMD:D_SOD-123" V 2100 3700 50  0001 C CNN
 F 3 "~" V 2100 3700 50  0001 C CNN
 	1    2100 3700
@@
 F 0 "C8" V 3325 3100 50  0000 C CNN
 F 1 "22u/TA" V 3416 3100 50  0000 C CNN
-F 2 "" H 3550 3100 50  0001 C CNN
+F 2 "Capacitor_Tantalum_SMD:CP_EIA-3216-18_Kemet-A" H 3550 3100 50  0001 C CNN
 F 3 "~" H 3550 3100 50  0001 C CNN
+F 4 "TAJA226K006RNJV" H 3550 3100 50  0001 C CNN "Partno"
 	1    3550 3100
 	0    1    1    0
@@
 F 0 "C9" H 3508 3654 50  0000 R CNN
 F 1 "10n" H 3508 3745 50  0000 R CNN
-F 2 "" H 3600 3700 50  0001 C CNN
+F 2 "Capacitor_SMD:C_0603_1608Metric" H 3600 3700 50  0001 C CNN
 F 3 "~" H 3600 3700 50  0001 C CNN
 	1    3600 3700
@@
 F 0 "H1" V 1400 6800 50  0000 L CNN
 F 1 "MountingHole_Pad" V 1500 6800 50  0000 L CNN
-F 2 "" H 1450 6600 50  0001 C CNN
+F 2 "Mounting_Holes:MountingHole_2.2mm_M2_ISO14580_Pad" H 1450 6600 50  0001 C CNN
 F 3 "~" H 1450 6600 50  0001 C CNN
 	1    1450 6600
@@
 F 0 "H2" V 1650 6800 50  0000 L CNN
 F 1 "MountingHole_Pad" V 1750 6800 50  0000 L CNN
-F 2 "" H 1700 6600 50  0001 C CNN
+F 2 "Mounting_Holes:MountingHole_2.2mm_M2_ISO14580_Pad" H 1700 6600 50  0001 C CNN
 F 3 "~" H 1700 6600 50  0001 C CNN
 	1    1700 6600
@@
 F 0 "H3" V 1900 6800 50  0000 L CNN
 F 1 "MountingHole_Pad" V 2000 6800 50  0000 L CNN
-F 2 "" H 1950 6600 50  0001 C CNN
+F 2 "Mounting_Holes:MountingHole_2.2mm_M2_ISO14580_Pad" H 1950 6600 50  0001 C CNN
 F 3 "~" H 1950 6600 50  0001 C CNN
 	1    1950 6600
@@
 F 0 "H4" V 2150 6800 50  0000 L CNN
 F 1 "MountingHole_Pad" V 2250 6800 50  0000 L CNN
-F 2 "" H 2200 6600 50  0001 C CNN
+F 2 "Mounting_Holes:MountingHole_2.2mm_M2_ISO14580_Pad" H 2200 6600 50  0001 C CNN
 F 3 "~" H 2200 6600 50  0001 C CNN
 	1    2200 6600
@@
 F 0 "C11" H 7742 2546 50  0000 L CNN
 F 1 "22u/TA" H 7742 2455 50  0000 L CNN
-F 2 "" H 7650 2500 50  0001 C CNN
+F 2 "Capacitor_Tantalum_SMD:CP_EIA-3216-18_Kemet-A" H 7650 2500 50  0001 C CNN
 F 3 "~" H 7650 2500 50  0001 C CNN
+F 4 "TAJA226K006RNJV" H 7650 2500 50  0001 C CNN "Partno"
 	1    7650 2500
 	1    0    0    -1
@@
 F 0 "C13" H 8242 2546 50  0000 L CNN
 F 1 "22u/TA" H 8242 2455 50  0000 L CNN
-F 2 "" H 8150 2500 50  0001 C CNN
+F 2 "Capacitor_Tantalum_SMD:CP_EIA-3216-18_Kemet-A" H 8150 2500 50  0001 C CNN
 F 3 "~" H 8150 2500 50  0001 C CNN
+F 4 "TAJA226K006RNJV" H 8150 2500 50  0001 C CNN "Partno"
 	1    8150 2500
 	1    0    0    -1
@@
 F 0 "C15" H 8742 2546 50  0000 L CNN
 F 1 "22u/TA" H 8742 2455 50  0000 L CNN
-F 2 "" H 8650 2500 50  0001 C CNN
+F 2 "Capacitor_Tantalum_SMD:CP_EIA-3216-18_Kemet-A" H 8650 2500 50  0001 C CNN
 F 3 "~" H 8650 2500 50  0001 C CNN
+F 4 "TAJA226K006RNJV" H 8650 2500 50  0001 C CNN "Partno"
 	1    8650 2500
 	1    0    0    -1
@@
 F 0 "C17" H 9242 2546 50  0000 L CNN
 F 1 "22u/TA" H 9242 2455 50  0000 L CNN
-F 2 "" H 9150 2500 50  0001 C CNN
+F 2 "Capacitor_Tantalum_SMD:CP_EIA-3216-18_Kemet-A" H 9150 2500 50  0001 C CNN
 F 3 "~" H 9150 2500 50  0001 C CNN
+F 4 "TAJA226K006RNJV" H 9150 2500 50  0001 C CNN "Partno"
 	1    9150 2500
 	1    0    0    -1
@@
 F 0 "C12" H 7742 3996 50  0000 L CNN
 F 1 "22u/TA" H 7742 3905 50  0000 L CNN
-F 2 "" H 7650 3950 50  0001 C CNN
+F 2 "Capacitor_Tantalum_SMD:CP_EIA-3216-18_Kemet-A" H 7650 3950 50  0001 C CNN
 F 3 "~" H 7650 3950 50  0001 C CNN
+F 4 "TAJA226K006RNJV" H 7650 3950 50  0001 C CNN "Partno"
 	1    7650 3950
 	1    0    0    -1
@@
 F 0 "C14" H 8242 3996 50  0000 L CNN
 F 1 "22u/TA" H 8242 3905 50  0000 L CNN
-F 2 "" H 8150 3950 50  0001 C CNN
+F 2 "Capacitor_Tantalum_SMD:CP_EIA-3216-18_Kemet-A" H 8150 3950 50  0001 C CNN
 F 3 "~" H 8150 3950 50  0001 C CNN
+F 4 "TAJA226K006RNJV" H 8150 3950 50  0001 C CNN "Partno"
 	1    8150 3950
 	1    0    0    -1
@@
 F 0 "C16" H 8742 3996 50  0000 L CNN
 F 1 "22u/TA" H 8742 3905 50  0000 L CNN
-F 2 "" H 8650 3950 50  0001 C CNN
+F 2 "Capacitor_Tantalum_SMD:CP_EIA-3216-18_Kemet-A" H 8650 3950 50  0001 C CNN
 F 3 "~" H 8650 3950 50  0001 C CNN
+F 4 "TAJA226K006RNJV" H 8650 3950 50  0001 C CNN "Partno"
 	1    8650 3950
 	1    0    0    -1
@@
 F 0 "C18" H 9242 3996 50  0000 L CNN
 F 1 "1u" H 9242 3905 50  0000 L CNN
-F 2 "" H 9150 3950 50  0001 C CNN
+F 2 "Capacitor_SMD:C_0603_1608Metric" H 9150 3950 50  0001 C CNN
 F 3 "~" H 9150 3950 50  0001 C CNN
 	1    9150 3950
@@
 F 0 "C19" H 9642 3996 50  0000 L CNN
 F 1 "10n" H 9642 3905 50  0000 L CNN
-F 2 "" H 9550 3950 50  0001 C CNN
+F 2 "Capacitor_SMD:C_0603_1608Metric" H 9550 3950 50  0001 C CNN
 F 3 "~" H 9550 3950 50  0001 C CNN
 	1    9550 3950
@@
 F 0 "C20" H 9992 3996 50  0000 L CNN
 F 1 "10n" H 9992 3905 50  0000 L CNN
-F 2 "" H 9900 3950 50  0001 C CNN
+F 2 "Capacitor_SMD:C_0603_1608Metric" H 9900 3950 50  0001 C CNN
 F 3 "~" H 9900 3950 50  0001 C CNN
 	1    9900 3950
@@
 F 0 "C10" H 5042 3646 50  0000 L CNN
 F 1 "100n" H 5042 3555 50  0000 L CNN
-F 2 "" H 4950 3600 50  0001 C CNN
+F 2 "Capacitor_SMD:C_0603_1608Metric" H 4950 3600 50  0001 C CNN
 F 3 "~" H 4950 3600 50  0001 C CNN
 	1    4950 3600
@@
 	6250 2700 3100 2700
 $Comp
-L Connector_Generic:Conn_01x02 J6
+L Mainboard-rescue:Conn_01x02-Connector_Generic J6
 U 1 1 5E2A6BF0
 P 2250 3250

Commit message: Add files via upload
assigned some more footprints
Parts:
- J5: footprint (none) -> Connector_PinHeader_2.54mm:PinHeader_1x03_P2.54mm_Vertical
- J6: footprint (none) -> Connector_PinHeader_2.54mm:PinHeader_1x02_P2.54mm_Vertical
- R6, R7: footprint (none) -> Resistor_SMD:R_0603_1608Metric
Changed lines of the file:
@@
 F 0 "J5" H 1418 3917 50  0000 C CNN
 F 1 "BATT" H 1418 3826 50  0000 C CNN
-F 2 "" H 1500 3600 50  0001 C CNN
+F 2 "Connector_PinHeader_2.54mm:PinHeader_1x03_P2.54mm_Vertical" H 1500 3600 50  0001 C CNN
 F 3 "~" H 1500 3600 50  0001 C CNN
 	1    1500 3600
@@
 F 0 "R6" H 3909 3346 50  0000 L CNN
 F 1 "9k1" H 3909 3255 50  0000 L CNN
-F 2 "" H 3850 3300 50  0001 C CNN
+F 2 "Resistor_SMD:R_0603_1608Metric" H 3850 3300 50  0001 C CNN
 F 3 "~" H 3850 3300 50  0001 C CNN
 	1    3850 3300
@@
 F 0 "R7" H 3909 3746 50  0000 L CNN
 F 1 "1k" H 3909 3655 50  0000 L CNN
-F 2 "" H 3850 3700 50  0001 C CNN
+F 2 "Resistor_SMD:R_0603_1608Metric" H 3850 3700 50  0001 C CNN
 F 3 "~" H 3850 3700 50  0001 C CNN
 	1    3850 3700
@@
 F 0 "J6" V 2214 3062 50  0000 R CNN
 F 1 "POT_PWR_SW" V 2123 3062 50  0000 R CNN
-F 2 "" H 2250 3250 50  0001 C CNN
+F 2 "Connector_PinHeader_2.54mm:PinHeader_1x02_P2.54mm_Vertical" H 2250 3250 50  0001 C CNN
 F 3 "~" H 2250 3250 50  0001 C CNN
 	1    2250 3250
