File: kicad/Mainboard/Modules.sch (KiCad schematic (older format))
At the start: 2 parts, among them U12 ESP-12F

Commit message: added ESP8266EX
Parts:
- removed U12: ESP-12F, RF_Module:ESP-12E, symbol ESP8266:ESP-12F
- added C100: 5p6, Capacitor_SMD:C_0603_1608Metric, symbol Device:C
- added C101, C103: 100n, Capacitor_SMD:C_0603_1608Metric, symbol Device:C
- added C102, C99: 10p, Capacitor_SMD:C_0603_1608Metric, symbol Device:C
- added R62: 12k, Resistor_SMD:R_0603_1608Metric, symbol Device:R
- added U12: GD25Q16CSIGTR, symbol Memory_Flash:W25Q32JVSS
- added U14: ESP8266EX, Package_DFN_QFN:QFN-32-1EP_5x5mm_P0.5mm_EP3.45x3.45mm, symbol MCU_Espressif:ESP8266EX
- added Y1: 24MHz, symbol Device:Crystal_GND24
Connections:
- net labels added: MEM_CLK, MEM_CS, MEM_D0, MEM_D1, MEM_D2, MEM_D3
- wire segments 11 -> 53
Other:
- moved on the sheet: C94
