File: kicad/Mainboard/Mainboard.sch (KiCad schematic (older format))
At the start: 0 parts

Commit message: Add files via upload
Changed lines of the file:
@@
 $Descr A4 11693 8268
 encoding utf-8
-Sheet 1 7
+Sheet 1 8
 Title "TR-9 Mainboard"
 Date ""
@@
 F1 "Connection.sch" 50
 $EndSheet
+$Sheet
+S 7000 850  1000 400
+U 5E25615D
+F0 "Modules" 50
+F1 "Modules.sch" 50
+$EndSheet
 $EndSCHEMATC
